File: Clock.sch (KiCad schematic (older format))
At the start: 0 parts

Commit message: Added clock and program counter modules.  Refined some schematics.
Parts:
- added C10, C11, C12, C13, C14, C4, C5, C6, C7, C8: 0.1u, symbol Device:C_Small
- added C9: 1u, symbol Device:C_Small
- added D3, D4: Blue, symbol Device:LED
- added D5: LED, symbol Device:LED
- added R10, R11, R4, R5, R7, R9: 4.7k, symbol Device:R
- added R3: 1M, symbol Device:R
- added R6: 3600, symbol Device:R
- added R8: 1800, symbol Device:R
- added RV1: 0-1.5M, symbol Device:R_POT
- added SW1: SW_Push, symbol Switch:SW_Push
- added SW2: SW_SPDT, symbol Switch:SW_SPDT
- added U2, U3, U4: LM555, symbol Timer:LM555
- added U5, U8, U9: 74LS04, symbol 74xx:74LS04
- added U6: 74LS08, symbol 74xx:74LS08
- added U7: 74LS32, symbol 74xx:74LS32
Connections:
- new net: C9.1, RV1.1, U2.2 (TR), U2.6 (THR)
- new net: C4.1, U2.5 (CV)
- new net: R6.2, R8.2, U2.7 (DIS)
- new net: R4.2, SW1.2, U4.2 (TR)
- new net: C10.1, U4.5 (CV)
- new net: C11.1, R3.2, U4.6 (THR), U4.7 (DIS)
- new net: SW2.1 (A), U3.2 (TR)
- new net: U3.3 (Q), U5.1, U6.2
- new net: R7.1, R9.2, SW2.3 (C), U3.4 (R)
- new net: C5.1, U3.5 (CV)
- new net: D3.2 (A), R11.2
- new net: R8.1, RV1.2
- new net: D4.2 (A), R5.2
- new net: U6.3, U7.1
- new net: U6.4, U7.3
- new net: U6.5, U8.2
- new net: U6.8, U7.2
- new net: U5.2, U6.9
- new net: D5.2 (A), R10.2
- new net Astable: R11.1, U2.3 (Q), U6.1
- new net CLK: R10.1, U6.6, U9.1
- new net GND: C10.2, C11.2, C12.2, C13.2, C14.2, C4.2, C5.2, C6.2, C7.2, C8.2, C9.2, D3.1 (K), D4.1 (K), D5.1 (K), SW1.1, SW2.2 (B), U2.1 (GND), U3.1 (GND), U3.6 (THR), U3.7 (DIS), U4.1 (GND), U5.7 (GND), U6.7 (GND), U7.7 (GND)
- new net HALT: U8.1
- new net Monostable: R5.1, U4.3 (Q), U6.10
- new net VCC: C12.1, C13.1, C14.1, C6.1, C7.1, C8.1, R3.1, R4.1, R6.1, R7.2, R9.1, U2.4 (R), U2.8 (VCC), U3.8 (VCC), U4.4 (R), U4.8 (VCC), U5.14 (VCC), U6.14 (VCC), U7.14 (VCC)
- new net ~CLK: U9.2
