File: ProgramCounter.sch (KiCad schematic (older format))
At the start: 0 parts

Commit message: Added clock and program counter modules.  Refined some schematics.
Parts:
- added C15, C16, C17: 0.1u, symbol Device:C_Small
- added D10, D11, D12, D13, D6, D7, D8, D9: Blue, symbol Device:LED
- added R12, R13, R14, R15, R16, R17, R18, R19: 4.7k, symbol Device:R
- added U10, U11: 74LS163, symbol 74xx:74LS163
- added U12: 74LS541, symbol 74xx:74LS541
Connections:
- new net: R15.2, U10.11 (Q3), U12.5 (A3)
- new net: R14.2, U10.12 (Q2), U12.4 (A2)
- new net: R13.2, U10.13 (Q1), U12.3 (A1)
- new net: R12.2, U10.14 (Q0), U12.2 (A0)
- new net: C15.1, U10.15 (TC), U11.2 (CP)
- new net: R19.2, U11.11 (Q3), U12.9 (A7)
- new net: R18.2, U11.12 (Q2), U12.8 (A6)
- new net: R17.2, U11.13 (Q1), U12.7 (A5)
- new net: R16.2, U11.14 (Q0), U12.6 (A4)
- new net: D6.2 (A), R12.1
- new net: D7.2 (A), R13.1
- new net: D8.2 (A), R14.1
- new net: D9.2 (A), R15.1
- new net: D10.2 (A), R16.1
- new net: D11.2 (A), R17.1
- new net: D12.2 (A), R18.1
- new net: D13.2 (A), R19.1
- new net B0: U10.3 (D0), U12.18 (Y0)
- new net B1: U10.4 (D1), U12.17 (Y1)
- new net B2: U10.5 (D2), U12.16 (Y2)
- new net B3: U10.6 (D3), U12.15 (Y3)
- new net B4: U11.3 (D0), U12.14 (Y4)
- new net B5: U11.4 (D1), U12.13 (Y5)
- new net B6: U11.5 (D2), U12.12 (Y6)
- new net B7: U11.6 (D3), U12.11 (Y7)
- new net GND: C15.2, C16.2, C17.2, D10.1 (K), D11.1 (K), D12.1 (K), D13.1 (K), D6.1 (K), D7.1 (K), D8.1 (K), D9.1 (K), U10.8 (GND), U11.8 (GND), U12.10 (GND)
- new net HALT: U11.15 (TC)
- new net PC_INC: U10.2 (CP)
- new net VCC: C16.1, C17.1, U10.10 (CET), U10.16 (VCC), U10.7 (CEP), U11.10 (CET), U11.16 (VCC), U11.7 (CEP), U12.20 (VCC)
- new net ~CLR: U10.1 (~MR), U11.1 (~MR)
- new net ~PC_LD: U10.9 (~PE), U11.9 (~PE)
- new net ~PC_OUT: U12.1 (G1), U12.19 (G2)
