File: ProgramCounter.sch (KiCad schematic (older format))
At the start: 47 parts, among them U801 74HCT08N, U802 74HCT74N, U803 74LS32, U804 74LS161AN, U805 74LS161AN, U806 74LS161AN, U807 74LS161AN, U808 74HCT541N, U809 74HCT541N

Commit message: Pre-removal of H/L byte deciding hardware
Connections:
- net labels added: ~PCH_IN, ~PCH_OUT, ~PCL_IN, ~PCL_OUT
- net labels removed: PC_IN, PC_OUT, ~CLK, ~PC_IN, ~PC_OUT
Other:
- moved on the sheet: U801A, U801B, U801C, U801D, U801E, U802A, U802B, U802C, U803A, U803B, U803C, U803D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

Commit message: Testing memory module
Parts:
- removed U801: 74HCT08N, symbol Breadboard_CPU-rescue:74LS08-74xx
- removed U802: 74HCT74N, symbol Breadboard_CPU-rescue:74LS74-74xx
- removed U803: 74LS32, symbol Breadboard_CPU-rescue:74LS32-74xx
Connections:
- net labels removed: ~PC_EN_LD_HIGH, ~PC_EN_LD_LOW, ~PC_EN_OUT_HIGH, ~PC_EN_OUT_LOW
- wire segments 282 -> 236
