File: ALU.sch (KiCad schematic (older format))
At the start: 0 parts

Commit message: Continued work.  Pushing for remote work.
Parts:
- added C37, C38, C39: 0.1u, symbol Device:C_Small
- added U32, U33: 74HC86, symbol 74xx:74HC86
- added U34, U35, U36: 74LS08, symbol 74xx:74LS08
- added U37, U39: 74HC283, symbol 74xx:74LS283
- added U38, U42: 74HC574, symbol 74xx:74HCT574
- added U40: 74HC138, symbol 74xx:74LS138
- added U41, U43: 74HCT541, symbol 74xx:74HCT541
Connections:
- new net: U39.1 (S2), U41.3 (A1)
- new net: U39.10 (S4), U41.5 (A3)
- new net: U33.3, U39.11 (B4)
- new net: U34.9, U38.16 (Q3), U39.12 (A4)
- new net: U39.13 (S3), U41.4 (A2)
- new net: U35.9, U38.17 (Q2), U39.14 (A3)
- new net: U33.6, U39.15 (B3)
- new net: U33.8, U39.2 (B2)
- new net: U34.12, U38.18 (Q1), U39.3 (A2)
- new net: U39.4 (S1), U41.2 (A0)
- new net: U35.12, U38.19 (Q0), U39.5 (A1)
- new net: U33.11, U39.6 (B1)
- new net: U37.7 (C0), U39.9 (C4)
- new net: U37.1 (S2), U41.7 (A5)
- new net: U37.10 (S4), U41.9 (A7)
- new net: U32.3, U37.11 (B4)
- new net: U35.1, U37.12 (A4), U38.12 (Q7)
- new net: U37.13 (S3), U41.8 (A6)
- new net: U36.1, U37.14 (A3), U38.13 (Q6)
- new net: U32.6, U37.15 (B3)
- new net: U32.8, U37.2 (B2)
- new net: U35.4, U37.3 (A2), U38.14 (Q5)
- new net: U37.4 (S1), U41.6 (A4)
- new net: U36.4, U37.5 (A1), U38.15 (Q4)
- new net: U32.11, U37.6 (B1)
- new net: U41.1 (G1), U41.19 (G2)
- new net: U41.11 (Y7), U42.9 (D7), U43.11 (Y7)
- new net: U41.12 (Y6), U42.8 (D6), U43.12 (Y6)
- new net: U41.13 (Y5), U42.7 (D5), U43.13 (Y5)
- new net: U41.14 (Y4), U42.6 (D4), U43.14 (Y4)
- new net: U41.15 (Y3), U42.5 (D3), U43.15 (Y3)
- new net: U41.16 (Y2), U42.4 (D2), U43.16 (Y2)
- new net: U41.17 (Y1), U42.3 (D1), U43.17 (Y1)
- new net: U41.18 (Y0), U42.2 (D0), U43.18 (Y0)
- new net: U43.1 (G1), U43.19 (G2)
- new net: U35.11, U43.2 (A0)
- new net: U34.11, U43.3 (A1)
- new net: U35.8, U43.4 (A2)
- new net: U34.8, U43.5 (A3)
- new net: U36.6, U43.6 (A4)
- new net: U35.6, U43.7 (A5)
- new net: U36.3, U43.8 (A6)
- new net: U35.3, U43.9 (A7)
- new net: U32.10, U32.13, U32.2, U32.5, U33.10, U33.13, U33.2, U33.5
- new net: U34.3, U38.11 (Cp)
- new net: U34.6, U42.11 (Cp)
- new net ALU_SAVE: U34.4
- new net B0: U33.12, U35.13, U38.2 (D0), U42.19 (Q0)
- new net B1: U33.9, U34.13, U38.3 (D1), U42.18 (Q1)
- new net B2: U33.4, U35.10, U38.4 (D2), U42.17 (Q2)
- new net B3: U33.1, U34.10, U38.5 (D3), U42.16 (Q3)
- new net B4: U32.12, U36.5, U38.6 (D4), U42.15 (Q4)
- new net B5: U32.9, U35.5, U38.7 (D5), U42.14 (Q5)
- new net B6: U32.4, U36.2, U38.8 (D6), U42.13 (Q6)
- new net B7: U32.1, U35.2, U38.9 (D7), U42.12 (Q7)
- new net CLK: U34.2, U34.5
- new net GND: C37.2, C38.2, C39.2, U37.8 (GND), U38.10 (GND), U39.8 (GND)
- new net OPC0: U40.1 (A0)
- new net OPC1: U40.2 (A1)
- new net OPC2: U40.3 (A2)
- new net OVERFLOW: U37.9 (C4)
- new net REGA_IN: U34.1
- new net VCC: C37.1, C38.1, C39.1, U37.16 (VCC), U38.20 (VCC), U39.16 (VCC)
- new net ~ALU_OUT: U42.1 (OE)
