File: ALU.sch (KiCad schematic (older format))
At the start: 15 parts, among them U32 74HC86, U33 74HC86, U34 74LS08, U35 74LS08, U36 74LS08, U37 74HC283, U38 74HC574, U39 74HC283, U40 74HC138, U41 74HCT541, U42 74HC574, U43 74HCT541

Commit message: Remote work
Parts:
- added C44, C45, C46, C47, C56, C57, C58, C59, C60: 0.1u, symbol Device:C_Small
- added R29, R30, R31, R35, R36, R37, R38, R39, R40, R41, R42: 10k, symbol Device:R
- added U46: 74HC05, symbol 74xx:74LS05
Connections:
- wire segments 253 -> 380
- no-connect marks 0 -> 6
Other:
- note added: "Cin\n"
- note added: "LS4b\n"
- note added: "MS4b\n"
- note added: "One or two args?"
- note added: "REGA may be high, low, or floating (output enable is inactive), \nso we must use pulldowns to force a low state default"
- moved on the sheet: U32E, U33E, U34B, U34E, U35E, U36E, U40, U42

Commit message: For desktop work
Parts:
- added U56: 74HC157, symbol 74xx:74LS157
Connections:
- net labels added: SEXT, argB6, argB7
- wire segments 380 -> 387
- no-connect marks 6 -> 12
Other:
- moved on the sheet: C56, C57, C58, C59, C60, U32E, U33E, U34E, U35E, U36E

Commit message: Migrated old device part numbers to SN74 LS or HCT series
Parts:
- removed R29, R30, R31: 10k, symbol Device:R
- removed U46: 74HC05, symbol 74xx:74LS05
- added U46: 74LS04, symbol 74xx:74LS04
- U32, U33: value 74HC86 -> 74LS86AN
- U34, U35, U36: value 74LS08 -> 74HCT08N
- U37, U39: value 74HC283 -> 74LS283N
- U38, U42: value 74HC574 -> 74HCT574N
- U40: value 74HC138 -> 74HCT138N
- U41, U43: value 74HCT541 -> 74HCT541N
- U56: value 74HC157 -> 74HCT157N
Connections:
- wire segments 387 -> 378
Other:
- moved on the sheet: C59, U36E

Commit message: Remote work
Parts:
- added C?: 0.1u, symbol Device:C_Small
Connections:
- net GND: now also U46.7 (GND), C?.2
- net VCC: now also U46.14 (VCC), C?.1
Other:
- note added: "8b Full Adders"
- note added: "ALU AND gate array"
- note added: "ALU Instruction Decoder"
- note added: "ALU Reg A"
- note added: "ALU output\nregister"
- note added: "Adder or AND\noperation buffers"
- note added: "Sign extender"
- note added: "XOR conditional inverters"
- moved on the sheet: U46G
Changed lines of the file:
@@
 L 74xx:74LS04 U?
 U 7 1 5FE38408
-P 15475 9375
+P 15450 8775
 AR Path="/5F05F116/5FE38408" Ref="U?"  Part="7"
 AR Path="/5EFC06D4/5FE38408" Ref="U46"  Part="7"
-F 0 "U46" H 15705 9421 50  0000 L CNN
-F 1 "74LS04" H 15705 9330 50  0000 L CNN
-F 2 "" H 15475 9375 50  0001 C CNN
-F 3 "http://www.ti.com/lit/gpn/sn74LS04" H 15475 9375 50  0001 C CNN
-	7    15475 9375
+F 0 "U46" H 15680 8821 50  0000 L CNN
+F 1 "74LS04" H 15680 8730 50  0000 L CNN
+F 2 "" H 15450 8775 50  0001 C CNN
+F 3 "http://www.ti.com/lit/gpn/sn74LS04" H 15450 8775 50  0001 C CNN
+	7    15450 8775
 	1    0    0    -1
 $EndComp
@@
 Wire Wire Line
 	5300 9900 7550 9900
+Text Notes 900  9375 0    118  ~ 0
+Sign extender
+Text Notes 1325 6175 0    118  ~ 0
+XOR conditional inverters
+Text Notes 5350 5725 0    118  ~ 0
+8b Full Adders
+Text Notes 9650 5200 0    118  ~ 0
+Adder or AND\noperation buffers
+Text Notes 11425 1650 0    118  ~ 0
+ALU output\nregister
+Text Notes 15375 7775 2    118  ~ 0
+ALU AND gate array
+$Comp
+L power:VCC #PWR?
+U 1 1 5F622F4C
+P 15450 8225
+AR Path="/5EFC09F3/5F622F4C" Ref="#PWR?"  Part="1"
+AR Path="/5F05F116/5F622F4C" Ref="#PWR?"  Part="1"
+AR Path="/5EFC06D4/5F622F4C" Ref="#PWR?"  Part="1"
+F 0 "#PWR?" H 15450 8075 50  0001 C CNN
+F 1 "VCC" H 15467 8398 50  0000 C CNN
+F 2 "" H 15450 8225 50  0001 C CNN
+F 3 "" H 15450 8225 50  0001 C CNN
+	1    15450 8225
+	1    0    0    -1
+$EndComp
+$Comp
+L power:GND #PWR?
+U 1 1 5F622F52
+P 15450 9325
+AR Path="/5EFC09F3/5F622F52" Ref="#PWR?"  Part="1"
+AR Path="/5F05F116/5F622F52" Ref="#PWR?"  Part="1"
+AR Path="/5EFC06D4/5F622F52" Ref="#PWR?"  Part="1"
+F 0 "#PWR?" H 15450 9075 50  0001 C CNN
+F 1 "GND" H 15455 9152 50  0000 C CNN
+F 2 "" H 15450 9325 50  0001 C CNN
+F 3 "" H 15450 9325 50  0001 C CNN
+	1    15450 9325
+	1    0    0    -1
+$EndComp
+$Comp
+L Device:C_Small C?
+U 1 1 5F622F58
+P 14800 8775
+AR Path="/5EFC09F3/5F622F58" Ref="C?"  Part="1"
+AR Path="/5F05F116/5F622F58" Ref="C?"  Part="1"
+AR Path="/5EFC06D4/5F622F58" Ref="C?"  Part="1"
+F 0 "C?" H 14892 8821 50  0000 L CNN
+F 1 "0.1u" H 14892 8730 50  0000 L CNN
+F 2 "" H 14800 8775 50  0001 C CNN
+F 3 "~" H 14800 8775 50  0001 C CNN
+	1    14800 8775
+	1    0    0    -1
+$EndComp
+Wire Wire Line
+	14800 8675 14800 8275
+Wire Wire Line
+	14800 8275 15450 8275
+Wire Wire Line
+	15450 8225 15450 8275
+Wire Wire Line
+	14800 8875 14800 9275
+Wire Wire Line
+	14800 9275 15450 9275
+Wire Wire Line
+	15450 9275 15450 9325
+Text Notes 6800 8625 0    118  ~ 0
+ALU Reg A
+Text Notes 8075 11125 0    118  ~ 0
+ALU Instruction Decoder
 $EndSCHEMATC

Commit message: Added ASSERT_ETI SR latch (NOR) - see timing diagram for int sheet
Parts:
- gave numbers to parts that had none: 1
Connections:
- net VCC: now also U56.10 (I1c), U56.11 (I0c), U56.13 (I1d), U56.14 (I0d)
- no-connect marks 12 -> 8
Changed lines of the file:
@@
 Text HLabel 2350 9100 0    50   Input ~ 0
 B5
-NoConn ~ 2350 9300
-NoConn ~ 2350 9400
-NoConn ~ 2350 9600
-NoConn ~ 2350 9700
 Wire Wire Line
 	2350 10000 2325 10000
@@
 L power:VCC #PWR0133
 U 1 1 607DC056
-P 2850 8350
-F 0 "#PWR0133" H 2850 8200 50  0001 C CNN
-F 1 "VCC" H 2865 8523 50  0000 C CNN
-F 2 "" H 2850 8350 50  0001 C CNN
-F 3 "" H 2850 8350 50  0001 C CNN
-	1    2850 8350
-	1    0    0    -1
-$EndComp
-Wire Wire Line
-	2850 8350 2850 8400
+P 2850 8300
+F 0 "#PWR0133" H 2850 8150 50  0001 C CNN
+F 1 "VCC" H 2865 8473 50  0000 C CNN
+F 2 "" H 2850 8300 50  0001 C CNN
+F 3 "" H 2850 8300 50  0001 C CNN
+	1    2850 8300
+	1    0    0    -1
+$EndComp
+Wire Wire Line
+	2850 8300 2850 8350
 Text HLabel 2325 9900 0    50   Input ~ 0
 SEXT
@@
 Wire Wire Line
 	5300 9900 7550 9900
-Text Notes 900  9375 0    118  ~ 0
+Text Notes 850  9375 0    118  ~ 0
 Sign extender
 Text Notes 1325 6175 0    118  ~ 0
@@
 AR Path="/5EFC09F3/5F622F4C" Ref="#PWR?"  Part="1"
 AR Path="/5F05F116/5F622F4C" Ref="#PWR?"  Part="1"
-AR Path="/5EFC06D4/5F622F4C" Ref="#PWR?"  Part="1"
-F 0 "#PWR?" H 15450 8075 50  0001 C CNN
+AR Path="/5EFC06D4/5F622F4C" Ref="#PWR0138"  Part="1"
+F 0 "#PWR0138" H 15450 8075 50  0001 C CNN
 F 1 "VCC" H 15467 8398 50  0000 C CNN
 F 2 "" H 15450 8225 50  0001 C CNN
@@
 AR Path="/5EFC09F3/5F622F52" Ref="#PWR?"  Part="1"
 AR Path="/5F05F116/5F622F52" Ref="#PWR?"  Part="1"
-AR Path="/5EFC06D4/5F622F52" Ref="#PWR?"  Part="1"
-F 0 "#PWR?" H 15450 9075 50  0001 C CNN
+AR Path="/5EFC06D4/5F622F52" Ref="#PWR0139"  Part="1"
+F 0 "#PWR0139" H 15450 9075 50  0001 C CNN
 F 1 "GND" H 15455 9152 50  0000 C CNN
 F 2 "" H 15450 9325 50  0001 C CNN
@@
 AR Path="/5EFC09F3/5F622F58" Ref="C?"  Part="1"
 AR Path="/5F05F116/5F622F58" Ref="C?"  Part="1"
-AR Path="/5EFC06D4/5F622F58" Ref="C?"  Part="1"
-F 0 "C?" H 14892 8821 50  0000 L CNN
+AR Path="/5EFC06D4/5F622F58" Ref="C63"  Part="1"
+F 0 "C63" H 14892 8821 50  0000 L CNN
 F 1 "0.1u" H 14892 8730 50  0000 L CNN
 F 2 "" H 14800 8775 50  0001 C CNN
@@
 Text Notes 8075 11125 0    118  ~ 0
 ALU Instruction Decoder
+Wire Wire Line
+	2850 8350 2150 8350
+Wire Wire Line
+	2150 8350 2150 9300
+Wire Wire Line
+	2150 9300 2350 9300
+Connection ~ 2850 8350
+Wire Wire Line
+	2850 8350 2850 8400
+Wire Wire Line
+	2350 9400 2150 9400
+Wire Wire Line
+	2150 9400 2150 9300
+Connection ~ 2150 9300
+Wire Wire Line
+	2150 9400 2150 9600
+Wire Wire Line
+	2150 9600 2350 9600
+Connection ~ 2150 9400
+Wire Wire Line
+	2150 9600 2150 9700
+Wire Wire Line
+	2150 9700 2350 9700
+Connection ~ 2150 9600
 $EndSCHEMATC

Commit message: Replaced all broken schematics with the up-to-date versions.  Some symbols missing.  This version will be the one created IRL except for the carry flag.
Parts:
- removed C46, C56, C57, C59: 0.1u, symbol Device:C_Small
- removed U34, U35, U36: 74HCT08N, symbol 74xx:74LS08
- removed U40: 74HCT138N, symbol 74xx:74LS138
- removed unit 5 of U46
- removed unit 6 of U46
- added C507, C510, C512, C513, C514, C515: 0.1u, symbol Breadboard_CPU-rescue:C_Small-Device
- added Q? (x2): Q_NPN_CBE, symbol Breadboard_CPU-rescue:Q_NPN_CBE-Device
- added R501, R502, R503, R505, R506, R508, R509, R511, R? (x3): 10k, symbol Breadboard_CPU-rescue:R-Device
- added U502, U503: 74HCT32N, symbol Breadboard_CPU-rescue:74LS32-74xx
- added unit 5 of U504
- added unit 6 of U504
- added U507: 74LS153, symbol 74xx:74LS153
- added U509, U513, U516: 74HCT08N, symbol Breadboard_CPU-rescue:74LS08-74xx
- added U517, U518: 74HCT74N, symbol Breadboard_CPU-rescue:74LS74-74xx
- C501: renamed from C37; symbol Device:C_Small -> Breadboard_CPU-rescue:C_Small-Device
- C502: renamed from C58; symbol Device:C_Small -> Breadboard_CPU-rescue:C_Small-Device
- C503: renamed from C38; symbol Device:C_Small -> Breadboard_CPU-rescue:C_Small-Device
- C504: renamed from C63; symbol Device:C_Small -> Breadboard_CPU-rescue:C_Small-Device
- C505: renamed from C39; symbol Device:C_Small -> Breadboard_CPU-rescue:C_Small-Device
- C506: renamed from C60; symbol Device:C_Small -> Breadboard_CPU-rescue:C_Small-Device
- C508: renamed from C44; symbol Device:C_Small -> Breadboard_CPU-rescue:C_Small-Device
- C509: renamed from C45; symbol Device:C_Small -> Breadboard_CPU-rescue:C_Small-Device
- C511: renamed from C47; symbol Device:C_Small -> Breadboard_CPU-rescue:C_Small-Device
- R504: renamed from R35; symbol Device:R -> Breadboard_CPU-rescue:R-Device
- R507: renamed from R36; symbol Device:R -> Breadboard_CPU-rescue:R-Device
- R510: renamed from R37; symbol Device:R -> Breadboard_CPU-rescue:R-Device
- R512: renamed from R38; symbol Device:R -> Breadboard_CPU-rescue:R-Device
- R513: renamed from R39; symbol Device:R -> Breadboard_CPU-rescue:R-Device
- R514: renamed from R40; symbol Device:R -> Breadboard_CPU-rescue:R-Device
- R515: renamed from R41; symbol Device:R -> Breadboard_CPU-rescue:R-Device
- R516: renamed from R42; symbol Device:R -> Breadboard_CPU-rescue:R-Device
- U501: renamed from U32; symbol 74xx:74HC86 -> Breadboard_CPU-rescue:74HC86-74xx
- U504: renamed from U46; symbol 74xx:74LS04 -> Breadboard_CPU-rescue:74LS04-74xx
- U505: renamed from U56; symbol 74xx:74LS157 -> Breadboard_CPU-rescue:74LS157-74xx
- U506: renamed from U33; symbol 74xx:74HC86 -> Breadboard_CPU-rescue:74HC86-74xx
- U508: renamed from U37; symbol 74xx:74LS283 -> Breadboard_CPU-rescue:74LS283-74xx
- U510: renamed from U38; symbol 74xx:74HCT574 -> Breadboard_CPU-rescue:74HCT574-74xx
- U511: renamed from U39; symbol 74xx:74LS283 -> Breadboard_CPU-rescue:74LS283-74xx
- U512: renamed from U41; symbol 74xx:74HCT541 -> Breadboard_CPU-rescue:74HCT541-74xx
- U514: renamed from U42; symbol 74xx:74HCT574 -> Breadboard_CPU-rescue:74HCT574-74xx
- U515: renamed from U43; symbol 74xx:74HCT541 -> Breadboard_CPU-rescue:74HCT541-74xx
Connections:
- net ALU_SAVE: now also U509.4
- net B0: now also U502.13, U513.13
- net B1: now also U502.12, U513.10
- net B2: now also U502.2, U513.5
- net B3: now also U502.1, U513.2
- net B4: now also U505.10 (I1c), U505.3 (I1a), U505.6 (I1b), U502.10, U516.13
- net B5: now also U505.2 (I0a), U502.9, U516.10; no longer U501.9, U505.3 (I1a), U505.6 (I1b)
- net B6: now also U510.8 (D6), U502.5
- net B7: now also U505.11 (I0c), U510.9 (D7), U502.4, U518.2 (D); no longer U505.2 (I0a)
- net CLK: now also R?.1, U509.10, U509.2, U509.5
- net GND: now also C507.2, C510.2, C512.2, C513.2, C514.2, C515.2, R501.2, R502.2, R503.2, R505.2, R506.2, R508.2, R509.2, R511.2, R?.2, U502.7 (GND), U503.7 (GND), U507.1 (Ea), U507.10 (I0b), U507.11 (I1b), U507.12 (I2b), U507.13 (I3b), U507.4 (I2a), U507.5 (I1a), U507.8 (GND), U509.7 (GND), U513.7 (GND), U517.7 (GND), U518.7 (GND)
- net VCC: now also C507.1, C510.1, C512.1, C513.1, C514.1, C515.1, Q?.1 (C), U502.14 (VCC), U503.14 (VCC), U507.15 (Eb), U507.16 (VCC), U509.14 (VCC), U513.14 (VCC), U517.10 (~S), U517.14 (VCC), U517.4 (~S), U518.10 (~S), U518.14 (VCC), U518.4 (~S); no longer U505.10 (I1c), U505.11 (I0c)
- net argB6: now also U516.5; no longer U510.8 (D6)
- net argB7: now also U505.9 (Zc), U507.14 (S0), U516.2; no longer U505.4 (Za), U510.9 (D7)
- net at R504.1, U510.19 (Q0), U511.5 (A1): now also U513.12
- net at R507.1, U510.18 (Q1), U511.3 (A2): now also U513.9
- net at R510.1, U510.17 (Q2), U511.14 (A3): now also U513.4
- net at R512.1, U510.16 (Q3), U511.12 (A4): now also U513.1
- net at R513.1, U508.5 (A1), U510.15 (Q4): now also U516.12
- net at R514.1, U508.3 (A2), U510.14 (Q5): now also U516.9
- net at R515.1, U508.14 (A3), U510.13 (Q6): now also U516.4
- net A[7]: now reaches R516.1, U508.12 (A4), U510.12 (Q7)
- net A[7]: now also U507.2 (S1), U516.1
- net ~UseANDs: now reaches U515.1 (G1), U515.19 (G2)
- net ~UseANDs: now also U504.12; no longer U504.2
- net ALU_USE_ADDERS: now reaches U504.3
- net at U511.7 (C0): now also U503.11; no longer U504.4
- net at U504.5: now also U503.8
- net ZFL: now reaches U504.6
- net ZFL: now also U518.12 (D), U518.9 (Q)
- net at U510.1 (OE): now also U504.2; no longer U504.8
- net C[7]: now reaches U504.9
- net C[7]: now also U512.11 (Y7), U514.9 (D7), U515.11 (Y7), R501.1, U507.6 (I0a)
- net at U512.12 (Y6), U514.8 (D6), U515.12 (Y6): now also R502.1
- net at U512.13 (Y5), U514.7 (D5), U515.13 (Y5): now also R503.1
- net at U512.14 (Y4), U514.6 (D4), U515.14 (Y4): now also R505.1
- net at U512.15 (Y3), U514.5 (D3), U515.15 (Y3): now also R506.1
- net at U512.16 (Y2), U514.4 (D2), U515.16 (Y2): now also R508.1
- net at U512.17 (Y1), U514.3 (D1), U515.17 (Y1): now also R509.1
- net at U512.18 (Y0), U514.2 (D0), U515.18 (Y0): now also R511.1
- net at U515.2 (A0): now also U513.11
- net at U515.3 (A1): now also U513.8
- net at U515.4 (A2): now also U513.6
- net at U515.5 (A3): now also U513.3
- net at U515.6 (A4): now also U516.11
- net at U515.7 (A5): now also U516.8
- net at U515.8 (A6): now also U516.6
- net at U515.9 (A7): now also U516.3
- net at U510.11 (Cp): now also U509.8
- net at U514.11 (Cp): now also U509.6, U517.11 (C)
- net OPC1 renamed ALU_INVERT_B
- net OPC2 renamed ~UseAdders
- net ~UseAdders: now also U504.4; no longer U504.1
- net OVERFLOW renamed CFL
- net CFL: now also U517.2 (D)
- net SEXT renamed ALU_SEXT_5
- net ~ALU_OUT: no longer names the net of U514.1 (OE)
- net ~ALU_OUT: now also U504.10
- new net: U509.3, U518.11 (C), U518.3 (C)
- new net: Q?.3 (E), R?.1, U517.3 (C)
- new net: U503.13, U509.11
- new net: U504.8, U507.3 (I3a)
- new net: Q?.2 (B), R?.2 (x2)
- new net: Q?.1 (C), Q?.3 (E)
- new net: U502.3, U503.1
- new net: U502.6, U503.2
- new net: U502.8, U503.4
- new net: U502.11, U503.5
- new net: U503.3, U503.9
- new net: U503.10, U503.6
- new net ALU_AREG_OUT: U504.1
- new net ALU_CFL_UPD: R?.1
- new net ALU_CIN: U503.12
- new net ALU_OUT: U504.11
- new net ALU_USE_ANDS: U504.13
- new net ALU_USE_CFL_SAVED: U509.12
- new net AREG_IN: U509.9
- new net CFL_SAVED: U509.13, U517.5 (Q)
- new net OFL: U507.7 (Za), U517.12 (D), U517.9 (Q)
- new net SFL: U518.5 (Q)
- new net UPDATE_CC: U509.1
- new net argB5: U501.9, U505.4 (Za)
- new net ~RST: U517.1 (~R), U517.13 (~R), U518.1 (~R), U518.13 (~R)
- no-connect marks 8 -> 6
Other:
- note removed: "ALU Instruction Decoder"
- note removed: "Cin\n"
- moved on the sheet: C501, C502, C503, C504, C505, C506, C508, C509, C511, R504, R507, R510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
