File: ALU.sch (KiCad schematic (older format))
At the start: 54 parts, among them U501 74LS86AN, U502 74HCT32N, U503 74HCT32N, U504 74LS04, U505 74HCT157N, U506 74LS86AN, U507 74LS153, U508 74LS283N, U509 74HCT08N, U510 74HCT574N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

Commit message: Added REGS_ASSERT_RS0.  Added user referenceable CFL to solve issue of performing arithmetic on stack frame and global pointers.  TRAP routines will be created to perform ADD operations (leveraging JC/JNC) on SFP and GP.  uCode rev. 1 created in GDrive.
Parts:
- added U601: 74HCT74N, symbol Breadboard_CPU-rescue:74LS74-74xx
- gave numbers to parts that had none: 5
Connections:
- net CFL: now also U601.12 (D), U601.9 (Q)
- net VCC: now also U601.10 (~S)
- net ~RST: now also U601.13 (~R)
- net at U509.11, U514.11 (Cp), U517.11 (C): now also U601.11 (C)
- no-connect marks 6 -> 7
Other:
- moved on the sheet: C501, C502, C503, C504, C505, C506, C507, C508, C509, C510, C511, C512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

Commit message: Testing memory module
Parts:
- removed U601: 74HCT74N, symbol Breadboard_CPU-rescue:74LS74-74xx
- added U650: ~, symbol Breadboard_CPU-rescue:74LS74-74xx
Connections:
- net CFL: now also U650.2 (D), U650.5 (Q)
- net VCC: now also U650.4 (~S)
- net ~RST: now also U650.1 (~R)
- net at U509.11, U514.11 (Cp), U517.11 (C): now also U650.3 (C)
Changed lines of the file:
@@
 	20650 7525 20650 7475
 NoConn ~ 20950 7275
-$Comp
-L Breadboard_CPU-rescue:74LS74-74xx U?
-U 2 1 60AE31EF
-P 20625 4825
-AR Path="/5F05F116/60AE31EF" Ref="U?"  Part="2"
-AR Path="/5EFC0970/60AE31EF" Ref="U?"  Part="2"
-AR Path="/5EFC0623/60AE31EF" Ref="U?"  Part="2"
-AR Path="/5EFC06D4/60AE31EF" Ref="U601"  Part="2"
-F 0 "U601" H 20425 5075 50  0000 C CNN
-F 1 "74HCT74N" H 20850 5075 50  0000 C CNN
-F 2 "" H 20625 4825 50  0001 C CNN
-F 3 "74xx/74hc_hct74.pdf" H 20625 4825 50  0001 C CNN
-	2    20625 4825
-	1    0    0    -1
-$EndComp
 Text HLabel 20625 5175 3    50   Input ~ 0
 ~RST
@@
 Wire Wire Line
 	19975 6125 20325 6125
+$Comp
+L Breadboard_CPU-rescue:74LS74-74xx U?
+U 1 1 69B2D25C
+P 20625 4825
+AR Path="/5EFC0970/69B2D25C" Ref="U?"  Part="1"
+AR Path="/5EFC0623/69B2D25C" Ref="U?"  Part="1"
+AR Path="/5EFC06D4/69B2D25C" Ref="U650"  Part="1"
+F 0 "U650" H 20825 5075 50  0000 C CNN
+F 1 "~" H 20375 5075 50  0000 C CNN
+F 2 "" H 20625 4825 50  0001 C CNN
+F 3 "74xx/74hc_hct74.pdf" H 20625 4825 50  0001 C CNN
+	1    20625 4825
+	1    0    0    -1
+$EndComp
 $EndSCHEMATC
