File: Memory.sch (KiCad schematic (older format))
At the start: 0 parts

Commit message: Continued work.  Pushing for remote work.
Parts:
- added C18, C40, C41: 1n, symbol Device:C_Small
- added C19, C28, C29, C30, C42, C43: 0.1u, symbol Device:C_Small
- added Q2, Q3, Q4: 2N2222, symbol Device:Q_NPN_CBE
- added R20, R21, R23, R24, R25, R26: 10k, symbol Device:R
- added R22: 470, symbol Device:R
- added R27, R28: 200, symbol Device:R
- added U13, U14: 74HC157, symbol 74xx:74LS157
- added U15: 74HC08, symbol 74xx:74LS08
- added U16: 74HC273, symbol 74xx:74AHCT273
- added U17: AS6C6264, symbol Memory:AS6C6264
- added U18, U19: AT28C64B, symbol Memory:AT28C64B
- added U36: 74LS08, symbol 74xx:74LS08
- added U44, U45: 74HC193, symbol 74xx:74LS193
Connections:
- new net: C18.2, Q2.1 (C), R22.1, U17.27 (~WE)
- new net: U15.3, U16.11 (Cp)
- new net: U44.12 (~CO), U45.5 (UP)
- new net: U44.13 (~BO), U45.4 (DOWN)
- new net: C41.2, Q4.1 (C), R28.1, U44.4 (DOWN)
- new net: C40.2, Q3.1 (C), R27.1, U44.5 (UP)
- new net: R20.1, U36.8
- new net: R21.1, U36.11
- new net: Q3.2 (B), R20.2
- new net: C41.1, R26.2
- new net: Q4.2 (B), R21.2
- new net: C18.1, R23.2
- new net: C40.1, R25.2
- new net: Q2.2 (B), R24.2
- new net: R24.1, U15.6
- new net A0: U13.4 (Za)
- new net A1: U13.7 (Zb)
- new net A2: U13.9 (Zc)
- new net A3: U13.12 (Zd)
- new net A4: U14.4 (Za)
- new net A5: U14.7 (Zb)
- new net A6: U14.9 (Zc)
- new net A7: U14.12 (Zd)
- new net B0: U16.3 (D0), U17.11 (DQ0)
- new net B1: U16.4 (D1), U17.12 (DQ1)
- new net B2: U16.7 (D2), U17.13 (DQ2)
- new net B3: U16.8 (D3), U17.15 (DQ3)
- new net B4: U16.13 (D4), U17.16 (DQ4)
- new net B5: U16.14 (D5), U17.17 (DQ5)
- new net B6: U16.17 (D6), U17.18 (DQ6)
- new net B7: U16.18 (D7), U17.19 (DQ7)
- new net CLK: U15.1, U15.5, U36.12, U36.9
- new net D0: U44.3 (QA)
- new net D1: U44.2 (QB)
- new net D2: U44.6 (QC)
- new net D3: U44.7 (QD)
- new net D4: U45.3 (QA)
- new net D5: U45.2 (QB)
- new net D6: U45.6 (QC)
- new net D7: U45.7 (QD)
- new net ETI_RTI: U13.1 (S), U14.1 (S), U17.1 (A14)
- new net GND: C19.1, C28.2, C29.2, C30.2, C42.1, C43.2, Q2.3 (E), Q3.3 (E), Q4.3 (E), U13.15 (E), U13.8 (GND), U14.15 (E), U14.8 (GND), U15.7 (GND), U16.10 (GND), U17.14 (Vss), U17.2 (A12), U17.20 (~CE), U17.21 (A10), U17.23 (A11), U17.24 (A9), U17.25 (A8), U17.26 (A13), U18.14 (GND), U18.20 (~CE), U18.21 (A10), U18.22 (~OE), U18.24 (A9), U18.25 (A8), U19.14 (GND), U19.2 (A12), U19.20 (~CE), U19.21 (A10), U19.22 (~OE), U19.24 (A9), U19.25 (A8), U44.8 (GND), U45.8 (GND)
- new net I0: U18.11 (I/O0)
- new net I1: U18.12 (I/O1)
- new net I10: U19.13 (I/O2)
- new net I11: U19.15 (I/O3)
- new net I12: U19.16 (I/O4)
- new net I13: U19.17 (I/O5)
- new net I14: U19.18 (I/O6)
- new net I15: U19.19 (I/O7)
- new net I2: U18.13 (I/O2)
- new net I3: U18.15 (I/O3)
- new net I4: U18.16 (I/O4)
- new net I5: U18.17 (I/O5)
- new net I6: U18.18 (I/O6)
- new net I7: U18.19 (I/O7)
- new net I8: U19.11 (I/O0)
- new net I9: U19.12 (I/O1)
- new net INTERRUPT: U18.23 (A11), U19.23 (A11)
- new net MAR_IN: U15.2
- new net MEM_IN: U15.4
- new net Q0: U13.2 (I0a)
- new net Q1: U13.5 (I0b)
- new net Q2: U13.11 (I0c)
- new net Q3: U13.14 (I0d)
- new net Q4: U14.2 (I0a)
- new net Q5: U14.5 (I0b)
- new net Q6: U14.11 (I0c)
- new net Q7: U14.14 (I0d)
- new net RST: U44.14 (CLR), U45.14 (CLR)
- new net STKPTR_DEC: U36.13
- new net STKPTR_INC: U36.10
- new net VCC: C19.2, C28.1, C29.1, C30.1, C42.2, C43.1, R22.2, R23.1, R25.1, R26.1, R27.2, R28.2, U13.16 (VCC), U14.16 (VCC), U15.14 (VCC), U16.20 (VCC), U17.28 (Vcc), U18.2 (A12), U18.27 (~WE), U18.28 (Vcc), U19.27 (~WE), U19.28 (Vcc), U44.11 (~LOAD), U44.16 (VCC), U45.11 (~LOAD), U45.16 (VCC)
- new net ~MEM_OUT: U17.22 (~OE)
- new net ~RST: U16.1 (~Mr)
- no-connect marks 0 -> 10
Other:
- note added: "EEPROM"
- note added: "SRAM"
