File: Registers.sch (KiCad schematic (older format))
At the start: 0 parts

Commit message: Continued work.  Pushing for remote work.
Parts:
- added C20, C21, C22, C23, C24, C25, C26, C27, C31, C32, C33, C34, C35, C36: 0.1u, symbol Device:C_Small
- added U20, U21, U22, U23, U24, U25, U26, U27: 74HC574, symbol 74xx:74HCT574
- added U29, U30, U31: 74HC27, symbol 74xx:74LS27
- added U5, U9: 74HC32, symbol 74xx:74LS32
- added U8: 74HC138, symbol 74xx:74LS138
Connections:
- new net: U20.1 (OE), U9.8
- new net: U20.11 (Cp), U29.12
- new net: U31.5, U5.9, U8.10 (O5)
- new net: U30.5, U5.12, U8.11 (O4)
- new net: U29.5, U8.12 (O3), U9.12
- new net: U31.13, U8.13 (O2), U9.1
- new net: U30.11, U8.14 (O1), U9.4
- new net: U29.13, U8.15 (O0), U9.9
- new net: U30.13, U5.1, U8.7 (O7)
- new net: U29.11, U5.4, U8.9 (O6)
- new net: U24.1 (OE), U9.6
- new net: U24.11 (Cp), U30.8
- new net: U21.1 (OE), U9.11
- new net: U21.11 (Cp), U29.6
- new net: U25.1 (OE), U5.11
- new net: U25.11 (Cp), U30.6
- new net: U22.1 (OE), U9.3
- new net: U22.11 (Cp), U31.12
- new net: U26.1 (OE), U5.8
- new net: U26.11 (Cp), U31.6
- new net: U23.1 (OE), U5.6
- new net: U23.11 (Cp), U29.8
- new net: U27.1 (OE), U5.3
- new net: U27.11 (Cp), U30.12
- new net B0: U20.19 (Q0), U20.2 (D0), U21.19 (Q0), U21.2 (D0), U22.19 (Q0), U22.2 (D0), U23.19 (Q0), U23.2 (D0), U24.19 (Q0), U24.2 (D0), U25.19 (Q0), U25.2 (D0), U26.19 (Q0), U26.2 (D0), U27.19 (Q0), U27.2 (D0)
- new net B1: U20.18 (Q1), U20.3 (D1), U21.18 (Q1), U21.3 (D1), U22.18 (Q1), U22.3 (D1), U23.18 (Q1), U23.3 (D1), U24.18 (Q1), U24.3 (D1), U25.18 (Q1), U25.3 (D1), U26.18 (Q1), U26.3 (D1), U27.18 (Q1), U27.3 (D1)
- new net B2: U20.17 (Q2), U20.4 (D2), U21.17 (Q2), U21.4 (D2), U22.17 (Q2), U22.4 (D2), U23.17 (Q2), U23.4 (D2), U24.17 (Q2), U24.4 (D2), U25.17 (Q2), U25.4 (D2), U26.17 (Q2), U26.4 (D2), U27.17 (Q2), U27.4 (D2)
- new net B3: U20.16 (Q3), U20.5 (D3), U21.16 (Q3), U21.5 (D3), U22.16 (Q3), U22.5 (D3), U23.16 (Q3), U23.5 (D3), U24.16 (Q3), U24.5 (D3), U25.16 (Q3), U25.5 (D3), U26.16 (Q3), U26.5 (D3), U27.16 (Q3), U27.5 (D3)
- new net B4: U20.15 (Q4), U20.6 (D4), U21.15 (Q4), U21.6 (D4), U22.15 (Q4), U22.6 (D4), U23.15 (Q4), U23.6 (D4), U24.15 (Q4), U24.6 (D4), U25.15 (Q4), U25.6 (D4), U26.15 (Q4), U26.6 (D4), U27.15 (Q4), U27.6 (D4)
- new net B5: U20.14 (Q5), U20.7 (D5), U21.14 (Q5), U21.7 (D5), U22.14 (Q5), U22.7 (D5), U23.14 (Q5), U23.7 (D5), U24.14 (Q5), U24.7 (D5), U25.14 (Q5), U25.7 (D5), U26.14 (Q5), U26.7 (D5), U27.14 (Q5), U27.7 (D5)
- new net B6: U20.13 (Q6), U20.8 (D6), U21.13 (Q6), U21.8 (D6), U22.13 (Q6), U22.8 (D6), U23.13 (Q6), U23.8 (D6), U24.13 (Q6), U24.8 (D6), U25.13 (Q6), U25.8 (D6), U26.13 (Q6), U26.8 (D6), U27.13 (Q6), U27.8 (D6)
- new net B7: U20.12 (Q7), U20.9 (D7), U21.12 (Q7), U21.9 (D7), U22.12 (Q7), U22.9 (D7), U23.12 (Q7), U23.9 (D7), U24.12 (Q7), U24.9 (D7), U25.12 (Q7), U25.9 (D7), U26.12 (Q7), U26.9 (D7), U27.12 (Q7), U27.9 (D7)
- new net GND: C20.2, C21.2, C22.2, C23.2, C24.2, C25.2, C26.2, C27.2, C31.2, C32.2, C33.2, C34.2, C35.2, C36.2, U20.10 (GND), U21.10 (GND), U22.10 (GND), U23.10 (GND), U24.10 (GND), U25.10 (GND), U26.10 (GND), U27.10 (GND), U29.7 (GND), U30.7 (GND), U31.7 (GND), U5.7 (GND), U8.4 (E1), U8.5 (E2), U8.8 (GND), U9.7 (GND)
- new net RS0: U8.1 (A0)
- new net RS1: U8.2 (A1)
- new net RS2: U8.3 (A2)
- new net VCC: C20.1, C21.1, C22.1, C23.1, C24.1, C25.1, C26.1, C27.1, C31.1, C32.1, C33.1, C34.1, C35.1, C36.1, U20.20 (VCC), U21.20 (VCC), U22.20 (VCC), U23.20 (VCC), U24.20 (VCC), U25.20 (VCC), U26.20 (VCC), U27.20 (VCC), U29.14 (VCC), U30.14 (VCC), U31.14 (VCC), U5.14 (VCC), U8.16 (VCC), U8.6 (E3), U9.14 (VCC)
- new net ~CLK: U29.1, U29.3, U29.9, U30.1, U30.3, U30.9, U31.1, U31.3
- new net ~REG_IN: U29.10, U29.2, U29.4, U30.10, U30.2, U30.4, U31.2, U31.4
- new net ~REG_OUT: U5.10, U5.13, U5.2, U5.5, U9.10, U9.13, U9.2, U9.5
Other:
- note added: "These bottom two probably aren't required"
