File: ConditionFlags.sch (KiCad schematic (older format))
At the start: 0 parts

Commit message: Finished int handler (CPU side) and started flags module
Parts:
- added U? (x2): 74HCT08N, symbol 74xx:74AHCT273
- added U?: 74HCT08N, symbol 74xx:74HCT541
- added U? (x5): 74HCT08N, symbol 74xx:74LS08
Changed lines of the file:
@@
 Comment4 ""
 $EndDescr
+$Comp
+L 74xx:74AHCT273 U?
+U 1 1 6038B6D8
+P 4100 2550
+AR Path="/5EFC0623/6038B6D8" Ref="U?"  Part="1"
+AR Path="/5F05F116/6038B6D8" Ref="U?"  Part="1"
+AR Path="/5EFC0970/6038B6D8" Ref="U?"  Part="1"
+F 0 "U?" H 4200 3300 50  0000 C CNN
+F 1 "74HCT08N" H 4325 3200 50  0000 C CNN
+F 2 "" H 4100 2550 50  0001 C CNN
+F 3 "https://assets.nexperia.com/documents/data-sheet/74AHC_AHCT273.pdf" H 4100 2550 50  0001 C CNN
+	1    4100 2550
+	1    0    0    -1
+$EndComp
+$Comp
+L 74xx:74AHCT273 U?
+U 1 1 6038BCDE
+P 3875 4175
+AR Path="/5EFC0623/6038BCDE" Ref="U?"  Part="1"
+AR Path="/5F05F116/6038BCDE" Ref="U?"  Part="1"
+AR Path="/5EFC0970/6038BCDE" Ref="U?"  Part="1"
+F 0 "U?" H 3975 4925 50  0000 C CNN
+F 1 "74HCT08N" H 4100 4825 50  0000 C CNN
+F 2 "" H 3875 4175 50  0001 C CNN
+F 3 "https://assets.nexperia.com/documents/data-sheet/74AHC_AHCT273.pdf" H 3875 4175 50  0001 C CNN
+	1    3875 4175
+	1    0    0    -1
+$EndComp
+$Comp
+L 74xx:74HCT541 U?
+U 1 1 6038DC95
+P 5550 3125
+AR Path="/5F05F116/6038DC95" Ref="U?"  Part="1"
+AR Path="/5EFC0970/6038DC95" Ref="U?"  Part="1"
+F 0 "U?" H 5625 3900 50  0000 C CNN
+F 1 "74HCT08N" H 5775 3800 50  0000 C CNN
+F 2 "" H 5550 3125 50  0001 C CNN
+F 3 "http://www.ti.com/lit/gpn/sn74HCT541" H 5550 3125 50  0001 C CNN
+	1    5550 3125
+	1    0    0    -1
+$EndComp
+$Comp
+L 74xx:74LS08 U?
+U 1 1 60397AAC
+P 7525 1250
+AR Path="/5EFC09F3/60397AAC" Ref="U?"  Part="1"
+AR Path="/5EFC0970/60397AAC" Ref="U?"  Part="1"
+F 0 "U?" H 7525 1575 50  0000 C CNN
+F 1 "74HCT08N" H 7525 1484 50  0000 C CNN
+F 2 "" H 7525 1250 50  0001 C CNN
+F 3 "http://www.ti.com/lit/gpn/sn74LS08" H 7525 1250 50  0001 C CNN
+	1    7525 1250
+	1    0    0    -1
+$EndComp
+$Comp
+L 74xx:74LS08 U?
+U 3 1 60397AB2
+P 7525 2150
+AR Path="/5EFC09F3/60397AB2" Ref="U?"  Part="3"
+AR Path="/5EFC0970/60397AB2" Ref="U?"  Part="3"
+F 0 "U?" H 7525 2475 50  0000 C CNN
+F 1 "74HCT08N" H 7525 2384 50  0000 C CNN
+F 2 "" H 7525 2150 50  0001 C CNN
+F 3 "http://www.ti.com/lit/gpn/sn74LS08" H 7525 2150 50  0001 C CNN
+	3    7525 2150
+	1    0    0    -1
+$EndComp
+$Comp
+L 74xx:74LS08 U?
+U 2 1 60399E27
+P 8000 1700
+AR Path="/5EFC09F3/60399E27" Ref="U?"  Part="2"
+AR Path="/5EFC0970/60399E27" Ref="U?"  Part="2"
+F 0 "U?" H 8000 2025 50  0000 C CNN
+F 1 "74HCT08N" H 8000 1934 50  0000 C CNN
+F 2 "" H 8000 1700 50  0001 C CNN
+F 3 "http://www.ti.com/lit/gpn/sn74LS08" H 8000 1700 50  0001 C CNN
+	2    8000 1700
+	1    0    0    -1
+$EndComp
+$Comp
+L 74xx:74LS08 U?
+U 5 1 603A09B7
+P 7450 3150
+AR Path="/5EFC09F3/603A09B7" Ref="U?"  Part="5"
+AR Path="/5EFC0970/603A09B7" Ref="U?"  Part="5"
+F 0 "U?" H 7680 3196 50  0000 L CNN
+F 1 "74HCT08N" H 7680 3105 50  0000 L CNN
+F 2 "" H 7450 3150 50  0001 C CNN
+F 3 "http://www.ti.com/lit/gpn/sn74LS08" H 7450 3150 50  0001 C CNN
+	5    7450 3150
+	1    0    0    -1
+$EndComp
+$Comp
+L 74xx:74LS08 U?
+U 4 1 603A2235
+P 8350 2625
+F 0 "U?" H 8350 2950 50  0000 C CNN
+F 1 "74HCT08N" H 8350 2859 50  0000 C CNN
+F 2 "" H 8350 2625 50  0001 C CNN
+F 3 "http://www.ti.com/lit/gpn/sn74LS08" H 8350 2625 50  0001 C CNN
+	4    8350 2625
+	1    0    0    -1
+$EndComp
 $EndSCHEMATC

Commit message: Pre non-interrupt split
Parts:
- removed U? (x2): 74HCT08N, symbol 74xx:74AHCT273
- removed U?: 74HCT08N, symbol 74xx:74HCT541
- added U65: 74HCT08N, symbol 74xx:74LS08
- added U66, U69, U70, U71: 74HCT74N, symbol 74xx:74LS74
- gave numbers to parts that had none: 1
