File: ControlUnit.sch (KiCad schematic (older format))
At the start: 21 parts

Commit message: Remote work
Parts:
- added U? (x2): 74HC244, symbol 74xx:74HC244
- gave numbers to parts that had none: 19
Connections:
- net labels added: CONDITION_STATUS, I2, INIT_INTERRUPT, OPC_0, OPC_1, OPC_2, OPC_3, RS0, RS1, RS2, uInst_0, uInst_1, uInst_2, uInst_3, ~0:2->RS, ~6:8->RS
- wire segments 147 -> 201
- no-connect marks 5 -> 7
Other:
- note added: "I0-2 only ever go to RS\nSame with I6-8\n\nI9-11 is the only special case"
- moved on the sheet: C49, C50, C51, C52, C53, C54, C55, U51, U52, U53, U54, U55

Commit message: For desktop work
Parts:
- added R67, R68, R69, R70, R71, R72, R73, R74, R75, R76, R77, R78, R79, R80, R81, R82, R83, R84, R85, R86, R87, R88, R89, R90, R91, R92, R93, R94, R95, R96, R97, R98, R? (x7): 10k, symbol Device:R
- added U62: 74HCT541, symbol 74xx:74HCT541
- added U63, U64, U65, U66: ULN2804A, symbol Transistor_Array:ULN2804A
- added U? (x7): 74HC05, symbol 74xx:74LS05
- gave numbers to parts that had none: 2
Connections:
- net labels added: ALU_SAVE, B0, B1, B2, B3, B4, B5, B6, B7, CC0, CC1, CC2, COND_IN, MAR_IN, MEM_IN, PC_INC, REGA_IN, SEXT, STKPTR_DEC, STKPTR_INC, ~0:7->BUS, ~9:11->CC, ~9:11->RS, ~ALU_OUT, ~MEM_OUT, ~PC_IN, ~PC_OUT, ~REG_IN, ~REG_OUT
- net labels removed: CONDITION_STATUS, i2
- wire segments 201 -> 484
- no-connect marks 7 -> 9
Other:
- moved on the sheet: C51, C52, C53, C54, C55, U51, U52, U53, U54, U55, U60, U61

Commit message: Migrated old device part numbers to SN74 LS or HCT series
Parts:
- removed R67, R68, R69, R70, R71, R72, R73, R74, R75, R76, R77, R78, R79, R80, R81, R82, R83, R84, R85, R86, R87, R88, R89, R90, R91, R92, R93, R94, R95, R96, R97, R98, R? (x7): 10k, symbol Device:R
- removed U63, U64, U65, U66: ULN2804A, symbol Transistor_Array:ULN2804A
- removed U? (x7): 74HC05, symbol 74xx:74LS05
- added C61, C62: 0.1u, symbol Device:C_Small
- added U57, U58: 74LS04, symbol 74xx:74LS04
- C52, C53, C54: value C_Small -> 0.1u
- U15, U47, U6: value 74HC08 -> 74HCT08N
- U48, U49: value 74HC574 -> 74HCT574N
- U50: value 74HC161 -> 74LS161AN
- U51: value 74HC157 -> 74HCT157N
- U60, U61: value 74HC244 -> 74HCT244N
- U62: value 74HCT541 -> 74HCT541N
Connections:
- net labels added: ETI_RTI, FINISH_INT, REF_INT, TR_HALT
- wire segments 484 -> 309
Other:
- moved on the sheet: C52, C53, C54, C55, U52, U53, U54, U55, U61, U62

Commit message: Remote work
Parts:
- removed U48, U49: 74HCT574N, symbol 74xx:74HCT574
- added C? (x5): 0.1u, symbol Device:C_Small
- added U48, U49: 74HCT273N, symbol 74xx:74AHCT273
- added U? (x2): 74HCT574N, symbol 74xx:74HCT574
- added U? (x5): 74HCT32N, symbol 74xx:74LS32
- added U? (x4): 74LS11, symbol 74xx:74LS11
- added U? (x3): 74HCT74N, symbol 74xx:74LS74
Connections:
- net labels added: END_ETI, FORCE_NO_INT, INT, INTC0, INTC1, INTC2, INTC3, ~INT_CODE_OUT, ~INT_DATA_OUT, ~INT_REQ, ~RST
- net labels removed: FINISH_INT, INIT_INTERRUPT
- wire segments 309 -> 389
- no-connect marks 9 -> 23
Other:
- note added: "Instruction Register"
- note added: "Instruction argument buffers"
- note added: "Interrupt\nStatus DFF"
- note added: "broken\n"
- note added: "uCode EEPROMs"
- note added: "uCode\nBinary Counter"
- moved on the sheet: C51, C52, C53, C54, C55, C61, C62, U15C, U47A, U47B, U47E, U51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

Commit message: Added ASSERT_ETI SR latch (NOR) - see timing diagram for int sheet
Parts:
- added C64: 0.1u, symbol Device:C_Small
- added U28, U59: 74LS04, symbol 74xx:74LS04
- added U? (x2): 74HCT02, symbol 74xx:74HCT02
- gave numbers to parts that had none: 10
Connections:
- net labels added: ASSERT_ETI, UNASSERT_ETI
- wire segments 389 -> 420
Other:
- note removed: "broken\n"
- moved on the sheet: U15C, U64D, U67A

Commit message: Finished int handler (CPU side) and started flags module
Parts:
- removed unit 4 of U64
- added C70: 0.1u, symbol Device:C_Small
- added unit 3 of U68
- gave numbers to parts that had none: 1
Connections:
- net labels added: FINISH_INT, INTD0, INTD1, INTD2, INTD3, INTD4, INTD5, INTD6, INTD7, RST
- wire segments 420 -> 452
- no-connect marks 23 -> 15
Other:
- moved on the sheet: C48, C62, C65, C66, C67, U15C, U28D, U28E, U28F, U47B, U50, U58G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

Commit message: Pre non-interrupt split
Parts:
- removed C66, C67: 0.1u, symbol Device:C_Small
- removed U65, U66: 74HCT574N, symbol 74xx:74HCT574
- removed unit 3 of U68
Connections:
- net CC0 is gone; now on net B0: U61.3 (2Y0)
- net CC1 is gone; now on net B1: U61.5 (2Y1)
- net CC2 is gone; now on net B2: U61.7 (2Y2)
- net ETI_RTI: now also U52.12 (I/O1); no longer U52.15 (I/O3)
- net FINISH_INT: now also U55.17 (I/O5); no longer U55.12 (I/O1)
- net I12: now also U51.2 (I0a); no longer U49.13 (D4)
- net I13: now also U51.5 (I0b); no longer U49.14 (D5)
- net I14: now also U51.11 (I0c); no longer U49.17 (D6)
- net I15: now also U51.14 (I0d); no longer U49.18 (D7)
- net IR_IN: now also U52.11 (I/O0); no longer U52.12 (I/O1)
- net OPC_0: now also U47.4, U49.12 (Q4); no longer U51.4 (Za)
- net OPC_1: now also U49.15 (Q5), U63.9; no longer U51.7 (Zb)
- net OPC_2: now also U49.16 (Q6), U63.10; no longer U51.9 (Zc)
- net OPC_3: now also U49.19 (Q7), U63.11; no longer U51.12 (Zd)
- net REF_INT: now also U55.16 (I/O4); no longer U55.19 (I/O7)
- net RST: now also U67.1 (~R)
- net STKPTR_DEC: now also U52.13 (I/O2); no longer U52.16 (I/O4)
- net STKPTR_INC: now also U52.15 (I/O3); no longer U52.17 (I/O5)
- net UNASSERT_ETI: now also U47.6; no longer U55.11 (I/O0)
- net at U59.3: now also U55.19 (I/O7); no longer U55.18 (I/O6)
- net at U59.1: now also U55.18 (I/O6); no longer U55.17 (I/O5)
- net at U63.8: now also U47.5
- net at U58.1: now also U52.17 (I/O5); no longer U52.11 (I/O0)
- net REGA_IN renamed ALU_REGA_IN
- net ~9:11->CC renamed ~9:11->BUS
- new net: U49.13 (D4), U51.4 (Za)
- new net: U49.14 (D5), U51.7 (Zb)
- new net: U49.17 (D6), U51.9 (Zc)
- new net: U49.18 (D7), U51.12 (Zd)
- new net PORT_A_IN: U55.11 (I/O0)
- new net PORT_B_IN: U55.12 (I/O1)
- new net UPDATE_CC: U52.16 (I/O4)
- no-connect marks 15 -> 9
Other:
- note added: "input"
- moved on the sheet: C50, C51, C70, U15C, U28D, U28E, U28F, U47B, U49, U51, U58A, U58B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

Commit message: Replaced all broken schematics with the up-to-date versions.  Some symbols missing.  This version will be the one created IRL except for the carry flag.
Parts:
- removed C51, C61, C62, C64, C65, C68, C69, C70: 0.1u, symbol Device:C_Small
- removed C55: C_Small, symbol Device:C_Small
- removed U15, U47, U6: 74HCT08N, symbol 74xx:74LS08
- removed U28, U57, U58, U59: 74LS04, symbol 74xx:74LS04
- removed U51: 74HCT157N, symbol 74xx:74LS157
- removed U55: AT28C64B, symbol Memory:AT28C64B
- removed U63: 74LS11, symbol 74xx:74LS11
- removed U64: 74HCT32N, symbol 74xx:74LS32
- removed U67: 74HCT74N, symbol 74xx:74LS74
- removed U68: 74HCT02, symbol 74xx:74HCT02
- added C601, C603, C606, C611, C612, C613, C614: 0.1u, symbol Breadboard_CPU-rescue:C_Small-Device
- added C610: C_Small, symbol Breadboard_CPU-rescue:C_Small-Device
- added U601, U604: 74HCT74N, symbol Breadboard_CPU-rescue:74LS74-74xx
- added U602: 74HCT08N, symbol Breadboard_CPU-rescue:74LS08-74xx
- added U603: 74LS153, symbol 74xx:74LS153
- added U613: AT28C64B, symbol Memory:AT28C64B
- added U615, U616: 74LS04, symbol Breadboard_CPU-rescue:74LS04-74xx
- C602: renamed from C48; symbol Device:C_Small -> Breadboard_CPU-rescue:C_Small-Device
- C604: renamed from C49; symbol Device:C_Small -> Breadboard_CPU-rescue:C_Small-Device
- C605: renamed from C50; symbol Device:C_Small -> Breadboard_CPU-rescue:C_Small-Device
- C607: renamed from C52; symbol Device:C_Small -> Breadboard_CPU-rescue:C_Small-Device
- C608: renamed from C53; symbol Device:C_Small -> Breadboard_CPU-rescue:C_Small-Device
- C609: renamed from C54; symbol Device:C_Small -> Breadboard_CPU-rescue:C_Small-Device
- U605: renamed from U60; symbol 74xx:74HC244 -> Breadboard_CPU-rescue:74HC244-74xx
- U606: renamed from U49; symbol 74xx:74AHCT273 -> Breadboard_CPU-rescue:74AHCT273-74xx
- U607: renamed from U48; symbol 74xx:74AHCT273 -> Breadboard_CPU-rescue:74AHCT273-74xx
- U608: renamed from U50; symbol 74xx:74LS163 -> Breadboard_CPU-rescue:74LS163-74xx
- U609: renamed from U61; symbol 74xx:74HC244 -> Breadboard_CPU-rescue:74HC244-74xx
- U614: renamed from U62; symbol 74xx:74HCT541 -> Breadboard_CPU-rescue:74HCT541-74xx
- renumbered U52 to U610, U53 to U611, U54 to U612
Connections:
- net labels added: ALU_AREG_OUT, ALU_CFL_UPD, ALU_CIN, ALU_INVERT_B, ALU_OUT, ALU_SEXT_5, ALU_USE_ADDERS, ALU_USE_ANDS, ALU_USE_CFL_SAVED, AREG_IN, COND_FL, IR_CLK, OFL, OPC_4, PC_IN, PC_OUT, SFL, SP_DEC, SP_IN, SP_INC, SP_OUT, ZFL, ~I[10:8]->BUS, ~I[10:8]->RS, ~I[7:0]->BUS, ~I[7:5]->RS, ~SP_IN, ~SP_OUT, ~sext(I[10:8])->BUS
- net labels removed: ALU_REGA_IN, ASSERT_ETI, COND_IN, ETI_RTI, FINISH_INT, I11, I12, I13, I14, I15, INT, PORT_A_IN, PORT_B_IN, REF_INT, RST, SEXT, STKPTR_DEC, STKPTR_INC, UNASSERT_ETI, ~0:2->RS, ~0:7->BUS, ~6:8->RS, ~9:11->BUS, ~9:11->RS, ~ALU_OUT, ~INT_CODE_OUT, ~INT_DATA_OUT, ~INT_REQ
- wire segments 393 -> 306
- no-connect marks 9 -> 5
Other:
- note added: "I11 - I15 contain the opcode\nI8 - I10 contain usually a register pointer or an immediate value\nI5 - I7 contain a second register sometimes\nI0 - I7 contains an immediate 8b value sometimes"
- note added: "This EEPROM should be \nclosest to the ALU"
- note removed: "I0-2 only ever go to RS\nSame with I6-8\n\nI9-11 is the only special case"
- note removed: "I12 - I15 contain the opcode\nI9 - I11 contain usually a register or some condition flags\nI6 - I8 contain a second register sometimes, same with I0 - I2\nI0 - I5/7 contain an offset or an immediate value (5 or 7 bits long)"
- note removed: "Interrupt\nStatus DFF"
- note removed: "input"
- moved on the sheet: C602, C604, C605, C607, C608, C609, U605, U606, U607, U608, U609, U610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
