File: PowerControl.sch (KiCad schematic (older format))
At the start: 9 parts, among them Q1 Q_PMOS_GDS, U1 LM1085-5.0

Commit message: Added clock and program counter modules.  Refined some schematics.
Connections:
- net Vo renamed VCC
- net Vs renamed VS
Changed lines of the file:
@@
 	0    1    1    0
 $EndComp
-Text GLabel 3250 2800 0    50   Input ~ 0
-Vs
 Wire Wire Line
 	3250 2800 3700 2800
@@
 Wire Wire Line
 	3900 3500 3900 3550
-Text GLabel 3300 3100 0    50   Input ~ 0
-GND
-Text GLabel 6550 2800 2    50   Input ~ 0
-Vo
 Wire Wire Line
 	6400 3500 6400 3550
@@
 Wire Wire Line
 	6400 2800 6550 2800
+$Comp
+L power:VS #PWR09
+U 1 1 5F035B21
+P 3250 2800
+F 0 "#PWR09" H 3050 2650 50  0001 C CNN
+F 1 "VS" V 3268 2928 50  0000 L CNN
+F 2 "" H 3250 2800 50  0001 C CNN
+F 3 "" H 3250 2800 50  0001 C CNN
+	1    3250 2800
+	0    -1   -1   0
+$EndComp
+$Comp
+L power:VCC #PWR010
+U 1 1 5F0366B6
+P 6550 2800
+F 0 "#PWR010" H 6550 2650 50  0001 C CNN
+F 1 "VCC" V 6567 2928 50  0000 L CNN
+F 2 "" H 6550 2800 50  0001 C CNN
+F 3 "" H 6550 2800 50  0001 C CNN
+	1    6550 2800
+	0    1    1    0
+$EndComp
+Text GLabel 3300 3100 0    50   Input ~ 0
+GND
 $EndSCHEMATC

Commit message: Replaced all broken schematics with the up-to-date versions.  Some symbols missing.  This version will be the one created IRL except for the carry flag.
Parts:
- C201: renamed from C1; symbol Device:C_Small -> Breadboard_CPU-rescue:C_Small-Device
- C202: renamed from C2; symbol Device:C_Small -> Breadboard_CPU-rescue:C_Small-Device
- C203: renamed from C3; symbol Device:C_Small -> Breadboard_CPU-rescue:C_Small-Device
- D201: renamed from D1; symbol Device:D_Zener -> Breadboard_CPU-rescue:D_Zener-Device
- D202: renamed from D2; symbol Device:LED -> Breadboard_CPU-rescue:LED-Device
- Q201: renamed from Q1; symbol Device:Q_PMOS_GDS -> Breadboard_CPU-rescue:Q_PMOS_GDS-Device
- R201: renamed from R1; symbol Device:R -> Breadboard_CPU-rescue:R-Device
- R202: renamed from R2; symbol Device:R -> Breadboard_CPU-rescue:R-Device
- U201: renamed from U1; symbol Regulator_Linear:LM1085-5.0 -> Breadboard_CPU-rescue:LM1085-5.0-Regulator_Linear
Changed lines of the file:
@@
 $Descr A4 11693 8268
 encoding utf-8
-Sheet 6 10
+Sheet 2 8
 Title ""
 Date ""
@@
 $EndDescr
 $Comp
-L Device:Q_PMOS_GDS Q1
+L Breadboard_CPU-rescue:Q_PMOS_GDS-Device Q201
 U 1 1 5EFC0CE7
 P 3900 2900
-F 0 "Q1" V 4242 2900 50  0000 C CNN
+F 0 "Q201" V 4242 2900 50  0000 C CNN
 F 1 "Q_PMOS_GDS" V 4151 2900 50  0000 C CNN
 F 2 "" H 4100 3000 50  0001 C CNN
@@
 $EndComp
 $Comp
-L Device:D_Zener D1
+L Breadboard_CPU-rescue:D_Zener-Device D201
 U 1 1 5EFC19F2
 P 4300 3000
-F 0 "D1" V 4254 3079 50  0000 L CNN
+F 0 "D201" V 4254 3079 50  0000 L CNN
 F 1 "10V" V 4345 3079 50  0000 L CNN
 F 2 "" H 4300 3000 50  0001 C CNN
@@
 	3250 2800 3700 2800
 $Comp
-L power:GND #PWR01
+L Breadboard_CPU-rescue:GND-power #PWR0202
 U 1 1 5EFC2D0B
 P 3450 3550
-F 0 "#PWR01" H 3450 3300 50  0001 C CNN
+F 0 "#PWR0202" H 3450 3300 50  0001 C CNN
 F 1 "GND" H 3455 3377 50  0000 C CNN
 F 2 "" H 3450 3550 50  0001 C CNN
@@
 	3450 3100 3450 3550
 $Comp
-L Device:R R1
+L Breadboard_CPU-rescue:R-Device R201
 U 1 1 5EFC37FA
 P 3900 3350
-F 0 "R1" H 3970 3396 50  0000 L CNN
+F 0 "R201" H 3970 3396 50  0000 L CNN
 F 1 "10k" H 3970 3305 50  0000 L CNN
 F 2 "" V 3830 3350 50  0001 C CNN
@@
 $EndComp
 $Comp
-L Regulator_Linear:LM1085-5.0 U1
+L Breadboard_CPU-rescue:LM1085-5.0-Regulator_Linear U201
 U 1 1 5EFC3C14
 P 5600 2800
-F 0 "U1" H 5600 3042 50  0000 C CNN
+F 0 "U201" H 5600 3042 50  0000 C CNN
 F 1 "LM1085-5.0" H 5600 2951 50  0000 C CNN
 F 2 "" H 5600 3050 50  0001 C CIN
@@
 $EndComp
 $Comp
-L Device:C_Small C1
+L Breadboard_CPU-rescue:C_Small-Device C201
 U 1 1 5EFC5530
 P 4900 3250
-F 0 "C1" H 4992 3296 50  0000 L CNN
+F 0 "C201" H 4992 3296 50  0000 L CNN
 F 1 "10u" H 4992 3205 50  0000 L CNN
 F 2 "" H 4900 3250 50  0001 C CNN
@@
 $EndComp
 $Comp
-L Device:C_Small C2
+L Breadboard_CPU-rescue:C_Small-Device C202
 U 1 1 5EFC61B4
 P 5600 3250
-F 0 "C2" H 5692 3296 50  0000 L CNN
+F 0 "C202" H 5692 3296 50  0000 L CNN
 F 1 "10u" H 5692 3205 50  0000 L CNN
 F 2 "" H 5600 3250 50  0001 C CNN
@@
 $EndComp
 $Comp
-L Device:C_Small C3
+L Breadboard_CPU-rescue:C_Small-Device C203
 U 1 1 5EFC64B7
 P 6000 3250
-F 0 "C3" H 6092 3296 50  0000 L CNN
+F 0 "C203" H 6092 3296 50  0000 L CNN
 F 1 "100u" H 6092 3205 50  0000 L CNN
 F 2 "" H 6000 3250 50  0001 C CNN
@@
 $EndComp
 $Comp
-L power:GND #PWR04
+L Breadboard_CPU-rescue:GND-power #PWR0205
 U 1 1 5EFC6BF9
 P 5600 3550
-F 0 "#PWR04" H 5600 3300 50  0001 C CNN
+F 0 "#PWR0205" H 5600 3300 50  0001 C CNN
 F 1 "GND" H 5605 3377 50  0000 C CNN
 F 2 "" H 5600 3550 50  0001 C CNN
@@
 $EndComp
 $Comp
-L power:GND #PWR05
+L Breadboard_CPU-rescue:GND-power #PWR0206
 U 1 1 5EFC748C
 P 6000 3550
-F 0 "#PWR05" H 6000 3300 50  0001 C CNN
+F 0 "#PWR0206" H 6000 3300 50  0001 C CNN
 F 1 "GND" H 6005 3377 50  0000 C CNN
 F 2 "" H 6000 3550 50  0001 C CNN
@@
 $EndComp
 $Comp
-L power:GND #PWR02
+L Breadboard_CPU-rescue:GND-power #PWR0203
 U 1 1 5EFC834C
 P 3900 3550
-F 0 "#PWR02" H 3900 3300 50  0001 C CNN
+F 0 "#PWR0203" H 3900 3300 50  0001 C CNN
 F 1 "GND" H 3905 3377 50  0000 C CNN
 F 2 "" H 3900 3550 50  0001 C CNN
@@
 $EndComp
 $Comp
-L power:GND #PWR03
+L Breadboard_CPU-rescue:GND-power #PWR0204
 U 1 1 5EFC8352
 P 4900 3550
-F 0 "#PWR03" H 4900 3300 50  0001 C CNN
+F 0 "#PWR0204" H 4900 3300 50  0001 C CNN
 F 1 "GND" H 4905 3377 50  0000 C CNN
 F 2 "" H 4900 3550 50  0001 C CNN
@@
 	6400 3150 6400 3200
 $Comp
-L power:GND #PWR06
+L Breadboard_CPU-rescue:GND-power #PWR0207
 U 1 1 5EFD7367
 P 6400 3550
-F 0 "#PWR06" H 6400 3300 50  0001 C CNN
+F 0 "#PWR0207" H 6400 3300 50  0001 C CNN
 F 1 "GND" H 6405 3377 50  0000 C CNN
 F 2 "" H 6400 3550 50  0001 C CNN
@@
 $EndComp
 $Comp
-L Device:R R2
+L Breadboard_CPU-rescue:R-Device R202
 U 1 1 5EFD633B
 P 6400 3350
-F 0 "R2" H 6470 3396 50  0000 L CNN
+F 0 "R202" H 6470 3396 50  0000 L CNN
 F 1 "4.7k" H 6470 3305 50  0000 L CNN
 F 2 "" V 6330 3350 50  0001 C CNN
@@
 $EndComp
 $Comp
-L Device:LED D2
+L Breadboard_CPU-rescue:LED-Device D202
 U 1 1 5EFD4D26
 P 6400 3000
-F 0 "D2" V 6439 2882 50  0000 R CNN
+F 0 "D202" V 6439 2882 50  0000 R CNN
 F 1 "Power" V 6348 2882 50  0000 R CNN
 F 2 "" H 6400 3000 50  0001 C CNN
@@
 	6400 2800 6550 2800
 $Comp
-L power:VS #PWR09
+L Breadboard_CPU-rescue:VS-power #PWR0201
 U 1 1 5F035B21
 P 3250 2800
-F 0 "#PWR09" H 3050 2650 50  0001 C CNN
+F 0 "#PWR0201" H 3050 2650 50  0001 C CNN
 F 1 "VS" V 3268 2928 50  0000 L CNN
 F 2 "" H 3250 2800 50  0001 C CNN
@@
 $EndComp
 $Comp
-L power:VCC #PWR010
+L Breadboard_CPU-rescue:VCC-power #PWR0208
 U 1 1 5F0366B6
 P 6550 2800
-F 0 "#PWR010" H 6550 2650 50  0001 C CNN
+F 0 "#PWR0208" H 6550 2650 50  0001 C CNN
 F 1 "VCC" V 6567 2928 50  0000 L CNN
 F 2 "" H 6550 2800 50  0001 C CNN
