File: Breadboard_CPU.sch (KiCad schematic (older format))
At the start: 21 parts, among them Q101 2N2222, SW101 RST

Commit message: Simulating negpulse
Changed lines of the file:
@@
 F8 "B6" B R 4200 6025 50
 F9 "B7" B R 4200 5925 50
-F10 "CLK" I L 3300 6450 50
+F10 "CLK" I L 3300 6550 50
 F11 "~MEM_OUT" I L 3300 6225 50
 F12 "MEM_IN" I L 3300 6325 50
 F13 "~RST" I L 3300 6725 50
-F14 "~CLK" I L 3300 6575 50
-F15 "MARH_IN" I L 3300 6025 50
-F16 "MARL_IN" I L 3300 6125 50
-F17 "MEM_RD_HB" I L 3300 5925 50
+F14 "MARH_IN" I L 3300 6025 50
+F15 "MARL_IN" I L 3300 6125 50
+F16 "MEM_RD_HB" I L 3300 5925 50
 $EndSheet
 $Sheet
@@
 Wire Wire Line
 	3300 6725 3250 6725
-Text GLabel 3250 6450 0    50   Input ~ 0
+Text GLabel 3250 6550 0    50   Input ~ 0
 CLK
 Wire Wire Line
-	3300 6450 3250 6450
+	3300 6550 3250 6550
 Text GLabel 6925 10025 2    50   Output ~ 0
 ~RST
@@
 Wire Wire Line
 	4200 3300 4875 3300
-Text GLabel 3250 6575 0    50   Input ~ 0
-~CLK
-Wire Wire Line
-	3250 6575 3300 6575
 $Sheet
 S 4875 2725 1125 3675
