File: KiCAD/Breadboard_CPU.sch (KiCad schematic (older format))
At the start: 21 parts, among them Q101 2N2222, SW101 RST

Commit message: Continued developing assembler
Changed lines of the file:
@@
 Wire Wire Line
 	6800 9600 6800 9675
-$Comp
-L Breadboard_CPU-rescue:GND-power #PWR0106
-U 1 1 5FCEEC34
-P 8775 3300
-F 0 "#PWR0106" H 8775 3050 50  0001 C CNN
-F 1 "GND" H 8780 3127 50  0000 C CNN
-F 2 "" H 8775 3300 50  0001 C CNN
-F 3 "" H 8775 3300 50  0001 C CNN
-	1    8775 3300
-	-1   0    0    -1
-$EndComp
-Wire Wire Line
-	9075 3275 8775 3275
-Wire Wire Line
-	8775 3275 8775 3300
 Text Notes 3300 10325 0    118  ~ 0
 Bus LEDs
 Wire Wire Line
-	8650 3175 9075 3175
-Wire Wire Line
-	8650 3175 8650 9350
-Wire Wire Line
-	8550 3075 9075 3075
+	8650 3075 9075 3075
+Wire Wire Line
+	8650 3075 8650 9350
 Wire Notes Line style solid
 	2225 1575 10350 1575
@@
 F4 "HALT_A" I L 9075 2975 50
 F5 "HALT_B" I L 9075 3075 50
-F6 "HALT_C" I L 9075 3175 50
-F7 "HALT_D" I L 9075 3275 50
 $EndSheet
 Text Notes 10925 5500 0    150  ~ 0
@@
 F13 "RS1" I R 4200 2925 50
 F14 "RS2" I R 4200 2825 50
-F15 "~RST" I L 3300 3875 50
-F16 "SP_INC" I R 4200 3400 50
-F17 "SP_DEC" I R 4200 3475 50
-F18 "RST" I L 3300 3750 50
-F19 "REG_ASSERT_RS0" I R 4200 3300 50
-F20 "SPL_IN" I L 3300 3125 50
-F21 "SPH_IN" I L 3300 3025 50
-F22 "SPL_OUT" I L 3300 2925 50
-F23 "CLK" I L 3300 3475 50
-F24 "SPH_OUT" I L 3300 2825 50
-F25 "~CLK" I L 3300 3600 50
+F15 "SP_INC" I R 4200 3400 50
+F16 "SP_DEC" I R 4200 3475 50
+F17 "REG_ASSERT_RS0" I R 4200 3300 50
+F18 "SPL_IN" I L 3300 3125 50
+F19 "SPH_IN" I L 3300 3025 50
+F20 "SPL_OUT" I L 3300 2925 50
+F21 "CLK" I L 3300 3475 50
+F22 "SPH_OUT" I L 3300 2825 50
+F23 "~CLK" I L 3300 3600 50
+F24 "RST" I L 3300 3750 50
 $EndSheet
 Wire Wire Line
@@
 F11 "~RST" I L 3300 5550 50
 F12 "CLK" I L 3300 5250 50
-F13 "TR_HALT" O L 3300 5150 50
-F14 "~CLK" I L 3300 5400 50
-F15 "~PCL_OUT" I L 3300 4825 50
-F16 "~PCL_IN" I L 3300 5025 50
-F17 "~PCH_IN" I L 3300 4925 50
-F18 "~PCH_OUT" I L 3300 4725 50
+F13 "~PCL_OUT" I L 3300 4825 50
+F14 "~PCL_IN" I L 3300 5025 50
+F15 "~PCH_IN" I L 3300 4925 50
+F16 "~PCH_OUT" I L 3300 4725 50
 $EndSheet
 Wire Wire Line
@@
 Wire Wire Line
 	6000 4425 6050 4425
-Text GLabel 3250 3875 0    50   Input ~ 0
-~RST
-Wire Wire Line
-	3300 3875 3250 3875
 Text GLabel 3250 3600 0    50   Input ~ 0
 ~CLK
@@
 Wire Wire Line
 	3300 5550 3250 5550
-Text GLabel 3250 5400 0    50   Input ~ 0
-~CLK
-Wire Wire Line
-	3250 5400 3300 5400
 Text GLabel 3250 5250 0    50   Input ~ 0
 CLK
@@
 	6450 9600 6450 9350
 Wire Wire Line
-	3300 5150 2925 5150
-Wire Wire Line
-	2925 5150 2925 8675
-Wire Wire Line
-	2925 8675 8550 8675
-Wire Wire Line
-	8550 8675 8550 3075
-Wire Wire Line
 	9075 2975 8450 2975
