File: KiCAD/Clock.sch (KiCad schematic (older format))
At the start: 33 parts, among them SW301 PULSE_CLK, SW302 TOG_SRC, U301 74HCT32N, U302 74LS04, U303 LM555, U304 LM555, U305 74HCT08N, U306 LM555

Commit message: Continued developing assembler
Parts:
- removed C310, C311: 0.1u, symbol Breadboard_CPU-rescue:C_Small-Device
- removed R307, R308: 10k, symbol Breadboard_CPU-rescue:R-Device
- removed R309: 100k, symbol Breadboard_CPU-rescue:R-Device
- removed SW302: TOG_SRC, symbol Breadboard_CPU-rescue:SW_Push-Switch
- removed U306: LM555, symbol Breadboard_CPU-rescue:LM555-Timer
- added R? (x3): 1k, symbol Device:R
- added U?: 74LS138, symbol 74xx:74LS138
Connections:
- net HALT_C is gone; now on an unnamed net: U301.12
- net CLK: now also U302.2; no longer U302.1, U305.11
- net GND: now also R?.2, R?.2, R?.2, U?.8 (GND)
- net HALT_A: now also U?.5 (E2); no longer U301.4
- net HALT_B: now also U?.4 (E1); no longer U301.5
- net VCC: now also U301.10, U301.9, U?.16 (VCC), U?.6 (E3)
- net ~CLK: now also U302.1, U302.4; no longer U302.2
- net at U302.5: now also U?.15 (O0); no longer U305.2
- net at U301.1: now also U301.6; no longer U305.3
- net at U301.2: now also U301.11; no longer U305.6
- net at U301.3: now also U302.3; no longer U305.12
- net at U301.8: no longer U302.3
- net at U302.6: now also U305.2; no longer U305.4
- net at U305.10: now also U302.8
- net CLK_IN_2: now reaches U305.9
- net at U305.13: now also U302.10; no longer U302.4
- net at U302.12: now also U305.5
- net at U302.13: now also U?.14 (O1)
- net at U302.11: now also U?.12 (O3)
- net at U302.9: now also U?.13 (O2)
- net Astable renamed CLK_IN_1
- net CLK_IN_1: now also U305.4; no longer U305.1
- net HALT_D: no longer names the net of U301.13
- net HALT_D: now also U305.11
- net Monostable renamed CLK_IN_0
- net CLK_IN_0: now also U305.1; no longer U305.5
- new net: U301.4, U305.3
- new net: U301.5, U305.6
- new net: R?.1, U?.3 (A2)
- new net CLK_IN_3: U305.12
- new net CLK_SEL_0: R?.1, U?.1 (A0)
- new net CLK_SEL_1: R?.1, U?.2 (A1)
- no-connect marks 10 -> 5
Other:
- note added: "Clock selector"
- note added: "Debounced button"
- note removed: "Astable or\nmonostable\nselector"
- note removed: "HALT logic"
- note removed: "Monostable button\npress"
- moved on the sheet: D303, R310, U301A, U301B, U301C, U301D, U302A, U302B, U302C, U302D, U302E, U302F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
