File: KiCAD/ControlUnit.sch (KiCad schematic (older format))
At the start: 30 parts, among them U602 74HCT08N, U603 74LS153, U605 74HCT244N, U606 74HCT273N, U607 74HCT273N, U608 74LS161AN, U609 74HCT244N, U610 AT28C64B, U611 AT28C64B, U612 AT28C64B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

Commit message: Continued developing assembler
Parts:
- U603: symbol 74xx:74LS153 -> Breadboard_CPU-rescue:74LS153-74xx
Connections:
- wire segments 305 -> 306
Changed lines of the file:
@@
 $EndComp
 NoConn ~ 3975 13125
-Text HLabel 3975 13425 2    50   Output ~ 0
+Text HLabel 3975 13225 2    50   Output ~ 0
 RS2
 Text HLabel 3975 13325 2    50   Output ~ 0
 RS1
-Text HLabel 3975 13225 2    50   Output ~ 0
+Text HLabel 3975 13425 2    50   Output ~ 0
 RS0
 Wire Wire Line
@@
 Text Label 5600 13775 2    50   ~ 0
 ~sext(I[10:8])->BUS
-Text Label 2975 13825 2    50   ~ 0
+Text Label 2975 13725 2    50   ~ 0
 ~I[10:8]->RS
-Text Label 2975 13025 2    50   ~ 0
+Text Label 2975 13225 2    50   ~ 0
 I7
-Text Label 2975 12925 2    50   ~ 0
+Text Label 2975 13325 2    50   ~ 0
 I6
-Text Label 2975 12825 2    50   ~ 0
+Text Label 2975 13425 2    50   ~ 0
 I5
 Text HLabel 3975 12825 2    50   Output ~ 0
@@
 Text HLabel 3975 13025 2    50   Output ~ 0
 RS2
-Text Label 2975 13425 2    50   ~ 0
+Text Label 2975 13025 2    50   ~ 0
 I10
-Text Label 2975 13325 2    50   ~ 0
+Text Label 2975 12925 2    50   ~ 0
 I9
-Text Label 2975 13225 2    50   ~ 0
+Text Label 2975 12825 2    50   ~ 0
 I8
-Text Label 2975 13725 2    50   ~ 0
+Text Label 2975 13825 2    50   ~ 0
 ~I[7:5]->RS
 Wire Wire Line
 	3475 12425 3475 12475
 $Comp
-L 74xx:74LS153 U603
+L Breadboard_CPU-rescue:74LS153-74xx U603
 U 1 1 61F73C07
 P 2725 8300
@@
 $EndComp
 Wire Wire Line
-	1325 8975 1325 8800
-Wire Wire Line
 	1325 9175 1325 9450
 $Comp
@@
 Wire Wire Line
 	2725 7250 2725 7300
-Wire Wire Line
-	2725 7250 1675 7250
 Text Label 3225 7600 0    50   ~ 0
 COND_FL
@@
 	11550 7850 11550 8200
 Wire Wire Line
-	2225 8100 1675 8100
-Wire Wire Line
-	1675 8100 1675 8300
-Wire Wire Line
 	2225 8300 1675 8300
 Connection ~ 1675 8300
@@
 Wire Wire Line
 	1675 8500 1675 8600
-Wire Wire Line
-	2225 8800 1325 8800
-Connection ~ 1325 8800
-Wire Wire Line
-	1325 8800 1325 7250
 Wire Wire Line
 	2225 8600 1675 8600
@@
 	15400 8150 15400 8550
 Text Label 2225 9100 2    50   ~ 0
+OPC_2
+Text Label 2225 9000 2    50   ~ 0
 OPC_1
-Text Label 2225 9000 2    50   ~ 0
-OPC_0
 Text HLabel 14125 14600 2    50   Output ~ 0
 ALU_CFL_UPD
@@
 NoConn ~ 14125 14100
 Wire Wire Line
-	1325 9450 2725 9450
-Wire Wire Line
-	1675 8100 1675 7250
-Connection ~ 1675 8100
+	1325 9450 1875 9450
+Wire Wire Line
+	1675 7250 1325 7250
+Wire Wire Line
+	2725 7250 1675 7250
 Connection ~ 1675 7250
 Wire Wire Line
-	1675 7250 1325 7250
+	1675 7250 1675 8300
+Wire Wire Line
+	1325 7250 1325 8975
+Wire Wire Line
+	1675 8600 1675 8800
+Wire Wire Line
+	1675 8800 2225 8800
+Connection ~ 1675 8600
+Wire Wire Line
+	2225 8100 1875 8100
+Wire Wire Line
+	1875 8100 1875 9450
+Connection ~ 1875 9450
+Wire Wire Line
+	1875 9450 2725 9450
 $EndSCHEMATC
