File: KiCAD/Memory.sch (KiCad schematic (older format))
At the start: 57 parts, among them Q401 2N2222, U402 74HCT08N, U403 74HCT08N, U404 74LS04, U407 74HCT138N, U408 74HCT74N, U409 74HCT273N, U410 74HCT273N, U412 AT28C64B, U415 74HCT574N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

Commit message: Restructured files.  Added EEPROM_Programming files.
Connections:
- wire segments 339 -> 347
- no-connect marks 6 -> 8
Other:
- moved on the sheet: U?A, U?D
Changed lines of the file:
@@
 L 74xx:74LS32 U?
 U 1 1 69626707
-P 20475 6825
-F 0 "U?" H 20475 7150 50  0000 C CNN
-F 1 "74HCT32" H 20475 7059 50  0000 C CNN
-F 2 "" H 20475 6825 50  0001 C CNN
-F 3 "http://www.ti.com/lit/gpn/sn74LS32" H 20475 6825 50  0001 C CNN
-	1    20475 6825
-	0    -1   -1   0
+P 19400 8225
+F 0 "U?" H 19400 8550 50  0000 C CNN
+F 1 "74HCT32" H 19400 8459 50  0000 C CNN
+F 2 "" H 19400 8225 50  0001 C CNN
+F 3 "http://www.ti.com/lit/gpn/sn74LS32" H 19400 8225 50  0001 C CNN
+	1    19400 8225
+	1    0    0    -1
 $EndComp
 $Comp
@@
 L 74xx:74LS32 U?
 U 4 1 6962BF2D
-P 19850 9050
-F 0 "U?" H 19850 9375 50  0000 C CNN
-F 1 "74HCT32" H 19850 9284 50  0000 C CNN
-F 2 "" H 19850 9050 50  0001 C CNN
-F 3 "http://www.ti.com/lit/gpn/sn74LS32" H 19850 9050 50  0001 C CNN
-	4    19850 9050
-	1    0    0    -1
+P 20475 6825
+F 0 "U?" H 20475 7150 50  0000 C CNN
+F 1 "74HCT32" H 20475 7059 50  0000 C CNN
+F 2 "" H 20475 6825 50  0001 C CNN
+F 3 "http://www.ti.com/lit/gpn/sn74LS32" H 20475 6825 50  0001 C CNN
+	4    20475 6825
+	0    -1   -1   0
 $EndComp
 $Comp
@@
 Wire Wire Line
 	11425 15300 11925 15300
+Wire Wire Line
+	19050 8075 19050 8125
+$Comp
+L Breadboard_CPU-rescue:VCC-power #PWR?
+U 1 1 60CDE0C4
+P 19050 8075
+F 0 "#PWR?" H 19050 7925 50  0001 C CNN
+F 1 "VCC" H 19067 8248 50  0000 C CNN
+F 2 "" H 19050 8075 50  0001 C CNN
+F 3 "" H 19050 8075 50  0001 C CNN
+	1    19050 8075
+	1    0    0    -1
+$EndComp
+Wire Wire Line
+	19050 8125 19100 8125
+Wire Wire Line
+	19050 8125 19050 8325
+Wire Wire Line
+	19050 8325 19100 8325
+Connection ~ 19050 8125
+Wire Wire Line
+	19050 8325 19050 8650
+Wire Wire Line
+	19050 8650 19100 8650
+Connection ~ 19050 8325
+Wire Wire Line
+	19050 8650 19050 8850
+Wire Wire Line
+	19050 8850 19100 8850
+Connection ~ 19050 8650
+NoConn ~ 19700 8225
+NoConn ~ 19700 8750
 Wire Bus Line
 	10000 2550 10000 13200

Commit message: Continued developing assembler
Parts:
- U? (x5): symbol 74xx:74LS32 -> Breadboard_CPU-rescue:74LS32-74xx
Changed lines of the file:
@@
 Text HLabel 11775 3150 2    50   BiDi ~ 0
 B0
-Text HLabel 2075 6400 3    50   Input ~ 0
+Text HLabel 2075 5700 1    50   Input ~ 0
 ~RST
 Wire Wire Line
-	2075 6400 2075 6350
+	2075 5700 2075 5750
 $Comp
 L Breadboard_CPU-rescue:VCC-power #PWR0401
 U 1 1 5F643852
-P 2075 5675
-F 0 "#PWR0401" H 2075 5525 50  0001 C CNN
-F 1 "VCC" H 2093 5848 50  0000 C CNN
-F 2 "" H 2075 5675 50  0001 C CNN
-F 3 "" H 2075 5675 50  0001 C CNN
-	1    2075 5675
-	-1   0    0    -1
-$EndComp
-Wire Wire Line
-	2075 5750 2075 5675
+P 2075 6425
+F 0 "#PWR0401" H 2075 6275 50  0001 C CNN
+F 1 "VCC" H 2093 6598 50  0000 C CNN
+F 2 "" H 2075 6425 50  0001 C CNN
+F 3 "" H 2075 6425 50  0001 C CNN
+	1    2075 6425
+	1    0    0    1
+$EndComp
+Wire Wire Line
+	2075 6350 2075 6425
 Wire Wire Line
 	2375 6050 2525 6050
@@
 $EndComp
 $Comp
-L 74xx:74LS32 U?
+L Breadboard_CPU-rescue:74LS32-74xx U?
 U 1 1 69626707
 P 19400 8225
@@
 $EndComp
 $Comp
-L 74xx:74LS32 U?
+L Breadboard_CPU-rescue:74LS32-74xx U?
 U 2 1 69628A06
 P 11725 4800
@@
 $EndComp
 $Comp
-L 74xx:74LS32 U?
+L Breadboard_CPU-rescue:74LS32-74xx U?
 U 3 1 6962A47E
 P 19400 8750
@@
 $EndComp
 $Comp
-L 74xx:74LS32 U?
+L Breadboard_CPU-rescue:74LS32-74xx U?
 U 4 1 6962BF2D
 P 20475 6825
@@
 $EndComp
 $Comp
-L 74xx:74LS32 U?
+L Breadboard_CPU-rescue:74LS32-74xx U?
 U 5 1 696316BF
 P 11925 14750
