File: KiCAD/PowerControl.sch (KiCad schematic (older format))
At the start: 9 parts, among them Q201 Q_PMOS_GDS, U201 LM1085-5.0

Commit message: Continued developing assembler
Parts:
- removed D201: 10V, symbol Breadboard_CPU-rescue:D_Zener-Device
Changed lines of the file:
@@
 	0    -1   -1   0
-$EndComp
-$Comp
-L Breadboard_CPU-rescue:D_Zener-Device D201
-U 1 1 5EFC19F2
-P 4300 3000
-F 0 "D201" V 4254 3079 50  0000 L CNN
-F 1 "10V" V 4345 3079 50  0000 L CNN
-F 2 "" H 4300 3000 50  0001 C CNN
-F 3 "~" H 4300 3000 50  0001 C CNN
-	1    4300 3000
-	0    1    1    0
 $EndComp
 Wire Wire Line
@@
 $EndComp
 Wire Wire Line
-	4100 2800 4300 2800
-Wire Wire Line
 	5900 2800 6000 2800
 Wire Wire Line
@@
 Wire Wire Line
 	4900 2800 5300 2800
-Wire Wire Line
-	3900 3150 3900 3100
-Wire Wire Line
-	3900 3150 4300 3150
-Wire Wire Line
-	4300 2850 4300 2800
-Connection ~ 4300 2800
-Wire Wire Line
-	4300 2800 4900 2800
-Wire Wire Line
-	3900 3150 3900 3200
-Connection ~ 3900 3150
 Wire Wire Line
 	3900 3500 3900 3550
@@
 Text GLabel 3300 3100 0    50   Input ~ 0
 GND
+Wire Wire Line
+	3900 3100 3900 3200
+Wire Wire Line
+	4100 2800 4900 2800
 $EndSCHEMATC
