File: KiCAD/ProgramCounter.sch (KiCad schematic (older format))
At the start: 44 parts, among them U804 74LS161AN, U805 74LS161AN, U806 74LS161AN, U807 74LS161AN, U808 74HCT541N, U809 74HCT541N

Commit message: Continued developing assembler
Connections:
- no-connect marks 0 -> 1
Changed lines of the file:
@@
 Wire Wire Line
 	10275 7525 10275 7575
+NoConn ~ 7550 9475
 $EndSCHEMATC
