File: KiCAD/Registers.sch (KiCad schematic (older format))
At the start: 72 parts, among them U701 74HCT138N, U702 74HCT08N, U704 74LS27, U705 74HCT32N, U706 74HCT574N, U707 74HCT574N, U708 74HCT574N, U710 74LS193, U711 74LS193, U712 74LS27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

Commit message: Edited SP async->sync converters to use BJT, C, 2R. Use DiLog for RS0|RS[0].
Parts:
- removed C? (x4): 0.1u, symbol Device:C_Small
- removed Q? (x2): Q_NPN_CBE, symbol Breadboard_CPU-rescue:Q_NPN_CBE-Device
- removed Q? (x4): Q_NPN_CBE, symbol Device:Q_NPN_CBE
- removed R? (x2): 10k, symbol Breadboard_CPU-rescue:R-Device
- removed R? (x4): 1, symbol Device:R
- removed R? (x8): 1k, symbol Device:R
- removed unit 4 of U702
- removed unit 2 of U702
- removed U? (x4): 74HCT08N, symbol Breadboard_CPU-rescue:74LS08-74xx
- removed U? (x4): 74LS04, symbol Breadboard_CPU-rescue:74LS04-74xx
- added C? (x4): 0.1u, symbol Breadboard_CPU-rescue:C_Small-Device
- added D? (x2): 1N4001, Diode_THT:D_DO-41_SOD81_P10.16mm_Horizontal, symbol Diode:1N4001
- added Q? (x4): 2N2222, symbol Breadboard_CPU-rescue:Q_NPN_CBE-Device
- added R? (x8): 1k, symbol Breadboard_CPU-rescue:R-Device
- added R? (x4): 100, symbol Breadboard_CPU-rescue:R-Device
- added unit 2 of U702
- added unit 4 of U702
- U702: value 74HCT08N -> 74LS08
Connections:
- wire segments 590 -> 563
Other:
- moved on the sheet: U702A, U702C

Commit message: Continued developing assembler
Parts:
- D? (x2): symbol Diode:1N4001 -> Breadboard_CPU-rescue:1N4001-Diode
- U702: symbol 74xx:74LS08 -> Breadboard_CPU-rescue:74LS08-74xx
Changed lines of the file:
@@
 $EndComp
 $Comp
-L Diode:1N4001 D?
+L Breadboard_CPU-rescue:1N4001-Diode D?
 U 1 1 60D096CA
 P 4125 4950
@@
 $EndComp
 $Comp
-L Diode:1N4001 D?
+L Breadboard_CPU-rescue:1N4001-Diode D?
 U 1 1 60D0C3EB
 P 4125 5275
@@
 	1425 11025 1475 11025
 $Comp
-L 74xx:74LS08 U702
+L Breadboard_CPU-rescue:74LS08-74xx U702
 U 2 1 63673E9D
 P 1775 8550
@@
 $EndComp
 $Comp
-L 74xx:74LS08 U702
+L Breadboard_CPU-rescue:74LS08-74xx U702
 U 4 1 636774E8
 P 3200 12775
