File: KiCAD/ALU.sch (KiCad schematic (older format))
At the start: 40 parts, among them Q501 Q_NPN_CBE, Q502 Q_NPN_CBE, U501 74LS86AN, U502 74HCT32N, U503 74HCT32N, U504 74LS04, U505 74HCT157N, U506 74LS86AN, U507 74LS153, U508 74LS283N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

Commit message: First working versiongit add .  Added CSU control signal for updating C and O flags during add operations only.  Added circuitry to disable the reg decoder unless ~RI or ~RO are asserted.  Potential future issues: PC clock noise, reg clock noise, clock module being crap..
Parts:
- R519: value 10k -> 1k
Connections:
- net at U509.11, U514.11 (Cp): no longer U517.11 (C), U650.3 (C)
- net UPDATE_CC renamed CCU
- new net CSU_CLK: U517.11 (C), U650.3 (C)
Changed lines of the file:
@@
 	1    0    0    -1
 $EndComp
-Wire Wire Line
-	16600 6125 19975 6125
 $Comp
 L Breadboard_CPU-rescue:74LS74-74xx U?
@@
 	19475 2600 19525 2600
 Text HLabel 19475 2600 0    50   Input ~ 0
-UPDATE_CC
+CCU
 Wire Wire Line
 	20125 2700 20175 2700
@@
 Wire Wire Line
 	15400 5650 15450 5650
-Connection ~ 16600 6125
 Wire Wire Line
 	19325 7675 19325 7625
@@
 P 19325 7875
 F 0 "R519" H 19395 7921 50  0000 L CNN
-F 1 "10k" H 19395 7830 50  0000 L CNN
+F 1 "1k" H 19395 7830 50  0000 L CNN
 F 2 "" V 19255 7875 50  0001 C CNN
 F 3 "~" H 19325 7875 50  0001 C CNN
@@
 Wire Wire Line
 	19975 4825 20325 4825
-Connection ~ 19975 6125
 Wire Wire Line
 	19975 6125 20325 6125
@@
 Wire Wire Line
 	12950 13450 12950 13400
+Text HLabel 19925 6125 0    50   Input ~ 0
+CSU_CLK
+Wire Wire Line
+	19925 6125 19975 6125
+Connection ~ 19975 6125
 $EndSCHEMATC
